Commit message: body design

File: body1.urdf (robot description, URDF)
Before this commit: robot robot, 10 links, 9 joints
Joints:
- joint Torso_BackLeg: origin xyz=0 -0.375 3 rpy=0 0 0 -> xyz=0 1.625 3 rpy=0 0 0
- joint Torso_BottomLeg: origin xyz=0 0 2.8 rpy=0 0 0 -> xyz=0 2 2.8 rpy=0 0 0
- joint Torso_FrontLeg: origin xyz=0 0.375 3 rpy=0 0 0 -> xyz=0 2.375 3 rpy=0 0 0
- joint Torso_LeftLeg: origin xyz=-0.375 0 3 rpy=0 0 0 -> xyz=-0.375 2 3 rpy=0 0 0
- joint Torso_RightLeg: origin xyz=0.375 0 3 rpy=0 0 0 -> xyz=0.375 2 3 rpy=0 0 0
- joint Torso_TopLeg: origin xyz=0 0 3.2 rpy=0 0 0 -> xyz=0 2 3.2 rpy=0 0 0

File: body2.urdf (robot description, URDF)
Before this commit: robot robot, 10 links, 9 joints
Joints:
- joint Torso_BackLeg: origin xyz=0 -0.375 3 rpy=0 0 0 -> xyz=2 -0.375 3 rpy=0 0 0
- joint Torso_BottomLeg: origin xyz=0 0 2.8 rpy=0 0 0 -> xyz=2 0 2.8 rpy=0 0 0
- joint Torso_FrontLeg: origin xyz=0 0.375 3 rpy=0 0 0 -> xyz=2 0.375 3 rpy=0 0 0
- joint Torso_LeftLeg: origin xyz=-0.375 0 3 rpy=0 0 0 -> xyz=1.625 0 3 rpy=0 0 0
- joint Torso_RightLeg: origin xyz=0.375 0 3 rpy=0 0 0 -> xyz=2.375 0 3 rpy=0 0 0
- joint Torso_TopLeg: origin xyz=0 0 3.2 rpy=0 0 0 -> xyz=2 0 3.2 rpy=0 0 0

File: body3.urdf (robot description, URDF)
Before this commit: robot robot, 10 links, 9 joints
Joints:
- joint Torso_BackLeg: origin xyz=0 -0.375 3 rpy=0 0 0 -> xyz=2 1.625 3 rpy=0 0 0
- joint Torso_BottomLeg: origin xyz=0 0 2.8 rpy=0 0 0 -> xyz=2 2 2.8 rpy=0 0 0
- joint Torso_FrontLeg: origin xyz=0 0.375 3 rpy=0 0 0 -> xyz=2 2.375 3 rpy=0 0 0
- joint Torso_LeftLeg: origin xyz=-0.375 0 3 rpy=0 0 0 -> xyz=1.625 2 3 rpy=0 0 0
- joint Torso_RightLeg: origin xyz=0.375 0 3 rpy=0 0 0 -> xyz=2.375 2 3 rpy=0 0 0
- joint Torso_TopLeg: origin xyz=0 0 3.2 rpy=0 0 0 -> xyz=2 2 3.2 rpy=0 0 0
