Commit message: begin converting to swarm

File: body0.urdf (robot description, URDF)
Before this commit: robot robot, 9 links, 8 joints
Links:
- link Torso: geometry collision box size=0.1 0.1 0.05; visual box size=0.1 0.1 0.05
Joints:
- joint Torso_BackLeg: origin xyz=0.0 -0.5 1.0 rpy=0 0 0 -> xyz=-3.0 -3.05 0.05 rpy=0 0 0
- joint Torso_FrontLeg: origin xyz=0.0 0.5 1.0 rpy=0 0 0 -> xyz=-3.0 -2.95 0.05 rpy=0 0 0

Commit message: fixed constants

File: body0.urdf (robot description, URDF)
Before this commit: robot robot, 9 links, 8 joints
Links:
- removed link BackLeg
- removed link BackLowerLeg
- removed link FrontLowerLeg
- removed link LeftLeg
- removed link LeftLowerLeg
- removed link RightLeg
- removed link RightLowerLeg
Joints:
- removed joint BackLeg_BackLowerLeg
- removed joint FrontLeg_FrontLowerLeg
- removed joint LeftLeg_LeftLowerLeg
- removed joint RightLeg_RightLowerLeg
- removed joint Torso_BackLeg
- removed joint Torso_LeftLeg
- removed joint Torso_RightLeg

Commit message: build spiral creature

File: body0.urdf (robot description, URDF)
Before this commit: robot robot, 2 links, 1 joints
Links:
- added link BackLeg, mass 1; collision box size=0.25 0.75 0.13333333333333333; visual box size=0.25 0.75 0.13333333333333333
- added link BottomLeg, mass 1; collision box size=0.1875 0.1875 0.8; visual box size=0.1875 0.1875 0.8
- added link BottomLowerLeg, mass 1; collision box size=0.1875 0.1875 0.6000000000000001; visual box size=0.1875 0.1875 0.6000000000000001
- added link LeftLeg, mass 1; collision box size=0.75 0.25 0.13333333333333333; visual box size=0.75 0.25 0.13333333333333333
- added link RightLeg, mass 1; collision box size=0.75 0.25 0.13333333333333333; visual box size=0.75 0.25 0.13333333333333333
- added link TopLeg, mass 1; collision box size=0.1875 0.1875 1.0; visual box size=0.1875 0.1875 1.0
- added link TopUpperLeg, mass 1; collision box size=0.1875 0.1875 0.6000000000000001; visual box size=0.1875 0.1875 0.6000000000000001
- link FrontLeg: geometry collision box size=0.25 0.75 0.13333333333333333; visual box size=0.25 0.75 0.13333333333333333
- link Torso: geometry collision box size=0.75 0.75 0.4; visual box size=0.75 0.75 0.4
Joints:
- added joint BottomLeg_BottomLowerLeg: type revolute, parent BottomLeg, child BottomLowerLeg, origin xyz=0 0 -0.8 rpy=0 0 0, axis 0 1 0, limit lower=-3.14159 upper=3.14159 effort=0.0 velocity=0.0
- added joint TopLeg_TopUpperLeg: type revolute, parent TopLeg, child TopUpperLeg, origin xyz=0 0 0.8 rpy=0 0 0, axis 0 1 0, limit lower=-3.14159 upper=3.14159 effort=0.0 velocity=0.0
- added joint Torso_BackLeg: type revolute, parent Torso, child BackLeg, origin xyz=-3 -3.375 1 rpy=0 0 0, axis 1 0 0, limit lower=-3.14159 upper=3.14159 effort=0.0 velocity=0.0
- added joint Torso_BottomLeg: type revolute, parent Torso, child BottomLeg, origin xyz=-3 -3 0.8 rpy=0 0 0, axis 0 1 0, limit lower=-3.14159 upper=3.14159 effort=0.0 velocity=0.0
- added joint Torso_LeftLeg: type revolute, parent Torso, child LeftLeg, origin xyz=-3.375 -3 1 rpy=0 0 0, axis 0 1 0, limit lower=-3.14159 upper=3.14159 effort=0.0 velocity=0.0
- added joint Torso_RightLeg: type revolute, parent Torso, child RightLeg, origin xyz=-2.625 -3 1 rpy=0 0 0, axis 0 1 0, limit lower=-3.14159 upper=3.14159 effort=0.0 velocity=0.0
- added joint Torso_TopLeg: type revolute, parent Torso, child TopLeg, origin xyz=-3 -3 1.2 rpy=0 0 0, axis 0 1 0, limit lower=-3.14159 upper=3.14159 effort=0.0 velocity=0.0
- joint Torso_FrontLeg: origin xyz=-3.0 -2.95 0.05 rpy=0 0 0 -> xyz=-3 -2.625 1 rpy=0 0 0

Commit message: Adjust camera position

File: body0.urdf (robot description, URDF)
Before this commit: robot robot, 9 links, 8 joints
Joints:
- joint Torso_BackLeg: origin xyz=-3 -3.375 1 rpy=0 0 0 -> xyz=-5 -5.375 1 rpy=0 0 0
- joint Torso_BottomLeg: origin xyz=-3 -3 0.8 rpy=0 0 0 -> xyz=-5 -5 0.8 rpy=0 0 0
- joint Torso_FrontLeg: origin xyz=-3 -2.625 1 rpy=0 0 0 -> xyz=-5 -4.625 1 rpy=0 0 0
- joint Torso_LeftLeg: origin xyz=-3.375 -3 1 rpy=0 0 0 -> xyz=-5.375 -5 1 rpy=0 0 0
- joint Torso_RightLeg: origin xyz=-2.625 -3 1 rpy=0 0 0 -> xyz=-4.625 -5 1 rpy=0 0 0
- joint Torso_TopLeg: origin xyz=-3 -3 1.2 rpy=0 0 0 -> xyz=-5 -5 1.2 rpy=0 0 0

Commit message: Change fitness function

File: body0.urdf (robot description, URDF)
Before this commit: robot robot, 10 links, 9 joints
Links:
- removed link FrontLowerLeg
- removed link TopUpperLeg
Joints:
- removed joint FrontLeg_FrontLowerLeg
- removed joint TopLeg_TopUpperLeg

File: body1.urdf (robot description, URDF)
Before this commit: robot robot, 10 links, 9 joints
Links:
- removed link FrontLowerLeg
- removed link TopUpperLeg
Joints:
- removed joint FrontLeg_FrontLowerLeg
- removed joint TopLeg_TopUpperLeg

File: body3.urdf (robot description, URDF)
Before this commit: robot robot, 10 links, 9 joints
Links:
- removed link FrontLowerLeg
- removed link TopUpperLeg
Joints:
- removed joint FrontLeg_FrontLowerLeg
- removed joint TopLeg_TopUpperLeg
- joint Torso_BackLeg: origin xyz=2 1.625 3 rpy=0 0 0 -> xyz=2 -0.375 3 rpy=0 0 0
- joint Torso_BottomLeg: origin xyz=2 2 2.8 rpy=0 0 0 -> xyz=2 0 2.8 rpy=0 0 0
- joint Torso_FrontLeg: origin xyz=2 2.375 3 rpy=0 0 0 -> xyz=2 0.375 3 rpy=0 0 0
- joint Torso_LeftLeg: origin xyz=1.625 2 3 rpy=0 0 0 -> xyz=1.625 0 3 rpy=0 0 0
- joint Torso_RightLeg: origin xyz=2.375 2 3 rpy=0 0 0 -> xyz=2.375 0 3 rpy=0 0 0
- joint Torso_TopLeg: origin xyz=2 2 3.2 rpy=0 0 0 -> xyz=2 0 3.2 rpy=0 0 0

File: body4.urdf (robot description, URDF)
Before this commit: robot robot, 8 links, 7 joints
Joints:
- joint Torso_BackLeg: origin xyz=0 3.625 3 rpy=0 0 0 -> xyz=2 1.625 3 rpy=0 0 0
- joint Torso_BottomLeg: origin xyz=0 4 2.8 rpy=0 0 0 -> xyz=2 2 2.8 rpy=0 0 0
- joint Torso_FrontLeg: origin xyz=0 4.375 3 rpy=0 0 0 -> xyz=2 2.375 3 rpy=0 0 0
- joint Torso_LeftLeg: origin xyz=-0.375 4 3 rpy=0 0 0 -> xyz=1.625 2 3 rpy=0 0 0
- joint Torso_RightLeg: origin xyz=0.375 4 3 rpy=0 0 0 -> xyz=2.375 2 3 rpy=0 0 0
- joint Torso_TopLeg: origin xyz=0 4 3.2 rpy=0 0 0 -> xyz=2 2 3.2 rpy=0 0 0

File: body5.urdf (robot description, URDF)
Before this commit: robot robot, 8 links, 7 joints
Joints:
- joint Torso_BackLeg: origin xyz=0 3.625 3 rpy=0 0 0 -> xyz=2 3.625 3 rpy=0 0 0
- joint Torso_BottomLeg: origin xyz=0 4 2.8 rpy=0 0 0 -> xyz=2 4 2.8 rpy=0 0 0
- joint Torso_FrontLeg: origin xyz=0 4.375 3 rpy=0 0 0 -> xyz=2 4.375 3 rpy=0 0 0
- joint Torso_LeftLeg: origin xyz=-0.375 4 3 rpy=0 0 0 -> xyz=1.625 4 3 rpy=0 0 0
- joint Torso_RightLeg: origin xyz=0.375 4 3 rpy=0 0 0 -> xyz=2.375 4 3 rpy=0 0 0
- joint Torso_TopLeg: origin xyz=0 4 3.2 rpy=0 0 0 -> xyz=2 4 3.2 rpy=0 0 0

File: body6.urdf (robot description, URDF)
Before this commit: robot robot, 8 links, 7 joints
Joints:
- joint Torso_BackLeg: origin xyz=0 3.625 3 rpy=0 0 0 -> xyz=4 -0.375 3 rpy=0 0 0
- joint Torso_BottomLeg: origin xyz=0 4 2.8 rpy=0 0 0 -> xyz=4 0 2.8 rpy=0 0 0
- joint Torso_FrontLeg: origin xyz=0 4.375 3 rpy=0 0 0 -> xyz=4 0.375 3 rpy=0 0 0
- joint Torso_LeftLeg: origin xyz=-0.375 4 3 rpy=0 0 0 -> xyz=3.625 0 3 rpy=0 0 0
- joint Torso_RightLeg: origin xyz=0.375 4 3 rpy=0 0 0 -> xyz=4.375 0 3 rpy=0 0 0
- joint Torso_TopLeg: origin xyz=0 4 3.2 rpy=0 0 0 -> xyz=4 0 3.2 rpy=0 0 0

File: body7.urdf (robot description, URDF)
Before this commit: robot robot, 8 links, 7 joints
Joints:
- joint Torso_BackLeg: origin xyz=0 3.625 3 rpy=0 0 0 -> xyz=4 1.625 3 rpy=0 0 0
- joint Torso_BottomLeg: origin xyz=0 4 2.8 rpy=0 0 0 -> xyz=4 2 2.8 rpy=0 0 0
- joint Torso_FrontLeg: origin xyz=0 4.375 3 rpy=0 0 0 -> xyz=4 2.375 3 rpy=0 0 0
- joint Torso_LeftLeg: origin xyz=-0.375 4 3 rpy=0 0 0 -> xyz=3.625 2 3 rpy=0 0 0
- joint Torso_RightLeg: origin xyz=0.375 4 3 rpy=0 0 0 -> xyz=4.375 2 3 rpy=0 0 0
- joint Torso_TopLeg: origin xyz=0 4 3.2 rpy=0 0 0 -> xyz=4 2 3.2 rpy=0 0 0

File: body8.urdf (robot description, URDF)
Before this commit: robot robot, 8 links, 7 joints
Joints:
- joint Torso_BackLeg: origin xyz=0 3.625 3 rpy=0 0 0 -> xyz=4 3.625 3 rpy=0 0 0
- joint Torso_BottomLeg: origin xyz=0 4 2.8 rpy=0 0 0 -> xyz=4 4 2.8 rpy=0 0 0
- joint Torso_FrontLeg: origin xyz=0 4.375 3 rpy=0 0 0 -> xyz=4 4.375 3 rpy=0 0 0
- joint Torso_LeftLeg: origin xyz=-0.375 4 3 rpy=0 0 0 -> xyz=3.625 4 3 rpy=0 0 0
- joint Torso_RightLeg: origin xyz=0.375 4 3 rpy=0 0 0 -> xyz=4.375 4 3 rpy=0 0 0
- joint Torso_TopLeg: origin xyz=0 4 3.2 rpy=0 0 0 -> xyz=4 4 3.2 rpy=0 0 0
