Commit message: all joints done from slides

File: body.urdf (robot description, URDF)
Before this commit: robot robot, 3 links, 2 joints
Links:
- added link Link3, mass 1; collision box size=1 1 1; visual box size=1 1 1
- added link Link4, mass 1; collision box size=1 1 1; visual box size=1 1 1
- added link Link5, mass 1; collision box size=1 1 1; visual box size=1 1 1
- added link Link6, mass 1; collision box size=1 1 1; visual box size=1 1 1
Joints:
- added joint Link2_Link3: type revolute, parent Link2, child Link3, origin xyz=0 0.5 0.5 rpy=0 0 0, axis 0 1 0, limit lower=-3.14159 upper=3.14159 effort=0.0 velocity=0.0
- added joint Link3_Link4: type revolute, parent Link3, child Link4, origin xyz=0 1 0 rpy=0 0 0, axis 0 1 0, limit lower=-3.14159 upper=3.14159 effort=0.0 velocity=0.0
- added joint Link4_Link5: type revolute, parent Link4, child Link5, origin xyz=0 0.5 -0.5 rpy=0 0 0, axis 0 1 0, limit lower=-3.14159 upper=3.14159 effort=0.0 velocity=0.0
- added joint Link5_Link6: type revolute, parent Link5, child Link6, origin xyz=0 0 -1 rpy=0 0 0, axis 0 1 0, limit lower=-3.14159 upper=3.14159 effort=0.0 velocity=0.0

Commit message: robot done

File: body.urdf (robot description, URDF)
Before this commit: robot robot, 7 links, 6 joints
Links:
- removed link Link0
- removed link Link1
- removed link Link2
- removed link Link3
- removed link Link4
- removed link Link5
- removed link Link6
- added link BackLeg, mass 1; collision box size=1 1 1; visual box size=1 1 1
- added link FrontLeg, mass 1; collision box size=1 1 1; visual box size=1 1 1
- added link Torso, mass 1; collision box size=1 1 1; visual box size=1 1 1
Joints:
- removed joint Link0_Link1
- removed joint Link1_Link2
- removed joint Link2_Link3
- removed joint Link3_Link4
- removed joint Link4_Link5
- removed joint Link5_Link6
- added joint Torso_BackLeg: type revolute, parent Torso, child BackLeg, origin xyz=0.5 0 1.0 rpy=0 0 0, axis 0 1 0, limit lower=-3.14159 upper=3.14159 effort=0.0 velocity=0.0
- added joint Torso_FrontLeg: type revolute, parent Torso, child FrontLeg, origin xyz=-0.5 0 1.0 rpy=0 0 0, axis 0 1 0, limit lower=-3.14159 upper=3.14159 effort=0.0 velocity=0.0

Commit message: up to step 45

File: body.urdf (robot description, URDF)
Before this commit: robot robot, 3 links, 2 joints
Links:
- added link LeftLeg, mass 1; collision box size=1 0.2 0.2; visual box size=1 0.2 0.2
- added link RightLeg, mass 1; collision box size=1 0.2 0.2; visual box size=1 0.2 0.2
- link BackLeg: geometry collision box size=0.2 1 0.2; visual box size=0.2 1 0.2
- link FrontLeg: geometry collision box size=0.2 1 0.2; visual box size=0.2 1 0.2
Joints:
- added joint Torso_LeftLeg: type revolute, parent Torso, child LeftLeg, origin xyz=-0.5 0.0 1.0 rpy=0 0 0, axis 0 1 0, limit lower=-3.14159 upper=3.14159 effort=0.0 velocity=0.0
- added joint Torso_RightLeg: type revolute, parent Torso, child RightLeg, origin xyz=0.5 0.0 1.0 rpy=0 0 0, axis 0 1 0, limit lower=-3.14159 upper=3.14159 effort=0.0 velocity=0.0
- joint Torso_BackLeg: axis 0 1 0 -> 1 0 0; origin xyz=0.5 0 1.0 rpy=0 0 0 -> xyz=0.0 -0.5 1.0 rpy=0 0 0
- joint Torso_FrontLeg: axis 0 1 0 -> 1 0 0; origin xyz=-0.5 0 1.0 rpy=0 0 0 -> xyz=0.0 0.5 1.0 rpy=0 0 0

Commit message: quad built

File: body.urdf (robot description, URDF)
Before this commit: robot robot, 5 links, 4 joints
Links:
- added link BackLowerLeg, mass 1; collision box size=0.2 0.2 1; visual box size=0.2 0.2 1
- added link FrontLowerLeg, mass 1; collision box size=0.2 0.2 1; visual box size=0.2 0.2 1
- added link LeftLowerLeg, mass 1; collision box size=0.2 0.2 1; visual box size=0.2 0.2 1
- added link RightLowerLeg, mass 1; collision box size=0.2 0.2 1; visual box size=0.2 0.2 1
Joints:
- added joint BackLeg_BackLowerLeg: type revolute, parent BackLeg, child BackLowerLeg, origin xyz=0.0 -1.0 0.0 rpy=0 0 0, axis 1 0 0, limit lower=-3.14159 upper=3.14159 effort=0.0 velocity=0.0
- added joint FrontLeg_FrontLowerLeg: type revolute, parent FrontLeg, child FrontLowerLeg, origin xyz=0.0 1.0 0.0 rpy=0 0 0, axis 1 0 0, limit lower=-3.14159 upper=3.14159 effort=0.0 velocity=0.0
- added joint LeftLeg_LeftLowerLeg: type revolute, parent LeftLeg, child LeftLowerLeg, origin xyz=-1.0 0.0 0.0 rpy=0 0 0, axis 0 1 0, limit lower=-3.14159 upper=3.14159 effort=0.0 velocity=0.0
- added joint RightLeg_RightLowerLeg: type revolute, parent RightLeg, child RightLowerLeg, origin xyz=1.0 0.0 0.0 rpy=0 0 0, axis 0 1 0, limit lower=-3.14159 upper=3.14159 effort=0.0 velocity=0.0

Commit message: left and right legs

File: body.urdf (robot description, URDF)
Before this commit: robot robot, 9 links, 8 joints
Links:
- removed link BackLeg
- removed link BackLowerLeg
- removed link FrontLeg
- removed link FrontLowerLeg
- removed link LeftLowerLeg
- removed link RightLowerLeg
- link LeftLeg: geometry collision box size=0.2 0.2 0.75; visual box size=0.2 0.2 0.75
- link RightLeg: geometry collision box size=0.2 0.2 0.75; visual box size=0.2 0.2 0.75
- link Torso: geometry collision box size=0.5 1.2 1.25; visual box size=0.5 1.2 1.25
Joints:
- removed joint BackLeg_BackLowerLeg
- removed joint FrontLeg_FrontLowerLeg
- removed joint LeftLeg_LeftLowerLeg
- removed joint RightLeg_RightLowerLeg
- removed joint Torso_BackLeg
- removed joint Torso_FrontLeg
- joint Torso_LeftLeg: origin xyz=-0.5 0.0 1.0 rpy=0 0 0 -> xyz=0 -0.25 0.75 rpy=0 0 0
- joint Torso_RightLeg: origin xyz=0.5 0.0 1.0 rpy=0 0 0 -> xyz=0 0.25 0.75 rpy=0 0 0

Commit message: build body

File: body.urdf (robot description, URDF)
Before this commit: robot robot, 3 links, 2 joints
Links:
- added link LeftArm, mass 1; collision box size=0.25 0.95 0.25; visual box size=0.25 0.95 0.25
- added link LeftFoot, mass 1; collision box size=0.75 0.3 0.1; visual box size=0.75 0.3 0.1
- added link LowerLeftArm, mass 1; collision box size=0.25 0.95 0.25; visual box size=0.25 0.95 0.25
- added link LowerLeftLeg, mass 1; collision box size=0.2 0.2 0.75; visual box size=0.2 0.2 0.75
- added link LowerRightArm, mass 1; collision box size=0.25 0.95 0.25; visual box size=0.25 0.95 0.25
- added link LowerRightLeg, mass 1; collision box size=0.2 0.2 0.75; visual box size=0.2 0.2 0.75
- added link RightArm, mass 1; collision box size=0.25 0.95 0.25; visual box size=0.25 0.95 0.25
- added link RightFoot, mass 1; collision box size=0.75 0.3 0.1; visual box size=0.75 0.3 0.1
Joints:
- added joint LeftArm_LowerLeftArm: type revolute, parent LeftArm, child LowerLeftArm, origin xyz=0.0 -0.95 0.0 rpy=0 0 0, axis 0 0 1, limit lower=-3.14159 upper=3.14159 effort=0.0 velocity=0.0
- added joint LowerLeftLeg_LeftFoot: type revolute, parent LowerLeftLeg, child LeftFoot, origin xyz=0.0 0.0 -0.75 rpy=0 0 0, axis 0 1 0, limit lower=-3.14159 upper=3.14159 effort=0.0 velocity=0.0
- added joint LowerRightLeg_RightFoot: type revolute, parent LowerRightLeg, child RightFoot, origin xyz=0.0 0.0 -0.75 rpy=0 0 0, axis 0 1 0, limit lower=-3.14159 upper=3.14159 effort=0.0 velocity=0.0
- added joint RightArm_LowerRightArm: type revolute, parent RightArm, child LowerRightArm, origin xyz=0.0 0.95 0.0 rpy=0 0 0, axis 0 0 1, limit lower=-3.14159 upper=3.14159 effort=0.0 velocity=0.0
- added joint Torso_LeftArm: type revolute, parent Torso, child LeftArm, origin xyz=0.0 -0.6 2.325 rpy=0 0 0, axis 1 0 0, limit lower=-3.14159 upper=3.14159 effort=0.0 velocity=0.0
- added joint Torso_LowerLeftLeg: type revolute, parent LeftLeg, child LowerLeftLeg, origin xyz=0.0 0.0 -0.75 rpy=0 0 0, axis 0 1 0, limit lower=-3.14159 upper=3.14159 effort=0.0 velocity=0.0
- added joint Torso_LowerRightLeg: type revolute, parent RightLeg, child LowerRightLeg, origin xyz=0.0 0.0 -0.75 rpy=0 0 0, axis 0 1 0, limit lower=-3.14159 upper=3.14159 effort=0.0 velocity=0.0
- added joint Torso_RightArm: type revolute, parent Torso, child RightArm, origin xyz=0.0 0.6 2.325 rpy=0 0 0, axis 1 0 0, limit lower=-3.14159 upper=3.14159 effort=0.0 velocity=0.0
- joint Torso_LeftLeg: origin xyz=0 -0.25 0.75 rpy=0 0 0 -> xyz=0 -0.25 1.6 rpy=0 0 0
- joint Torso_RightLeg: origin xyz=0 0.25 0.75 rpy=0 0 0 -> xyz=0 0.25 1.5 rpy=0 0 0

Commit message: hinge loss function

File: body.urdf (robot description, URDF)
Before this commit: robot robot, 11 links, 10 joints
Links:
- removed link LeftArm
- removed link RightArm
- added link LeftArmX, mass 1; collision box size=0 0 0; visual box size=0 0 0
- added link LeftArmZ, mass 1; collision box size=0.25 0.95 0.25; visual box size=0.25 0.95 0.25
- added link RightArmX, mass 1; collision box size=0 0 0; visual box size=0 0 0
- added link RightArmZ, mass 1; collision box size=0.25 0.95 0.25; visual box size=0.25 0.95 0.25
Joints:
- removed joint LeftArm_LowerLeftArm
- removed joint RightArm_LowerRightArm
- removed joint Torso_LeftArm
- removed joint Torso_RightArm
- added joint LeftArmX_LeftArmZ: type revolute, parent LeftArmX, child LeftArmZ, origin xyz=0.0 0.0 0.0 rpy=0 0 0, axis 0 0 1, limit lower=-3.14159 upper=3.14159 effort=0.0 velocity=0.0
- added joint LeftArmZ_LowerLeftArm: type revolute, parent LeftArmZ, child LowerLeftArm, origin xyz=0.0 -0.95 0.0 rpy=0 0 0, axis 0 0 1, limit lower=-3.14159 upper=3.14159 effort=0.0 velocity=0.0
- added joint RightArmX_RightArmZ: type revolute, parent RightArmX, child RightArmZ, origin xyz=0.0 0 0 rpy=0 0 0, axis 0 0 1, limit lower=-3.14159 upper=3.14159 effort=0.0 velocity=0.0
- added joint RightArmZ_LowerRightArm: type revolute, parent RightArmZ, child LowerRightArm, origin xyz=0.0 0.95 0.0 rpy=0 0 0, axis 0 0 1, limit lower=-3.14159 upper=3.14159 effort=0.0 velocity=0.0
- added joint Torso_LeftArmX: type revolute, parent Torso, child LeftArmX, origin xyz=0.0 -0.6 2.325 rpy=0 0 0, axis 1 0 0, limit lower=-3.14159 upper=3.14159 effort=0.0 velocity=0.0
- added joint Torso_RightArmX: type revolute, parent Torso, child RightArmX, origin xyz=0.0 0.6 2.325 rpy=0 0 0, axis 1 0 0, limit lower=-3.14159 upper=3.14159 effort=0.0 velocity=0.0

Commit message: final

File: body.urdf (robot description, URDF)
Before this commit: robot robot, 13 links, 12 joints
Joints:
- joint Torso_RightLeg: origin xyz=0 0.25 1.5 rpy=0 0 0 -> xyz=0 0.25 1.6 rpy=0 0 0
