Commit message: color sensors

File: body.urdf (robot description, URDF)
Before this commit: robot robot, 4 links, 3 joints
Links:
- removed link Link0Link11
- added link Link10, mass 1; collision box size=0.289894209378449 0.3440572245439849 0.5033246164770036; visual box size=0.289894209378449 0.3440572245439849 0.5033246164770036
- added link Link10Link110, mass 1; collision box size=0 0 0; visual box size=0 0 0
- added link Link11, mass 1; collision box size=0.23048929422978615 0.7230499624108918 0.98868263266242; visual box size=0.23048929422978615 0.7230499624108918 0.98868263266242
- added link Link11Link120, mass 1; collision box size=0 0 0; visual box size=0 0 0
- added link Link12, mass 1; collision box size=0.6145624339903446 0.5030481387881167 0.9075291404269014; visual box size=0.6145624339903446 0.5030481387881167 0.9075291404269014
- added link Link12Link130, mass 1; collision box size=0 0 0; visual box size=0 0 0
- added link Link12Link131, mass 1; collision box size=0 0 0; visual box size=0 0 0
- added link Link13, mass 1; collision box size=0.08471743299549728 0.7066246726596259 0.7885625348151296; visual box size=0.08471743299549728 0.7066246726596259 0.7885625348151296
- added link Link13Link140, mass 1; collision box size=0 0 0; visual box size=0 0 0
- added link Link14, mass 1; collision box size=0.11919983767429032 0.9429736253086106 0.7841487564903633; visual box size=0.11919983767429032 0.9429736253086106 0.7841487564903633
- added link Link14Link150, mass 1; collision box size=0 0 0; visual box size=0 0 0
- added link Link14Link151, mass 1; collision box size=0 0 0; visual box size=0 0 0
- added link Link15, mass 1; collision box size=0.11866247091310489 0.6057533568110886 0.5752147305041113; visual box size=0.11866247091310489 0.6057533568110886 0.5752147305041113
- added link Link16, mass 1; collision box size=0.21761440909753382 0.5518196335360861 0.14972787713119928; visual box size=0.21761440909753382 0.5518196335360861 0.14972787713119928
- added link Link16Link170, mass 1; collision box size=0 0 0; visual box size=0 0 0
- added link Link16Link171, mass 1; collision box size=0 0 0; visual box size=0 0 0
- added link Link17, mass 1; collision box size=0.8055139515221608 0.3840055679952633 0.2239342210932017; visual box size=0.8055139515221608 0.3840055679952633 0.2239342210932017
- added link Link17Link180, mass 1; collision box size=0 0 0; visual box size=0 0 0
- added link Link17Link181, mass 1; collision box size=0 0 0; visual box size=0 0 0
- added link Link18, mass 1; collision box size=0.34667811060666387 0.42962978375535 0.7253250815261304; visual box size=0.34667811060666387 0.42962978375535 0.7253250815261304
- added link Link18Link190, mass 1; collision box size=0 0 0; visual box size=0 0 0
- added link Link18Link191, mass 1; collision box size=0 0 0; visual box size=0 0 0
- added link Link19, mass 1; collision box size=0.7267461245100323 0.7999117653558807 0.5689834804723336; visual box size=0.7267461245100323 0.7999117653558807 0.5689834804723336
- added link Link1Link20, mass 1; collision box size=0 0 0; visual box size=0 0 0
- added link Link1Link21, mass 1; collision box size=0 0 0; visual box size=0 0 0
- added link Link2, mass 1; collision box size=0.6364123475017288 0.23912236519631302 0.06556436989900005; visual box size=0.6364123475017288 0.23912236519631302 0.06556436989900005
- added link Link2Link30, mass 1; collision box size=0 0 0; visual box size=0 0 0
- added link Link3, mass 1; collision box size=0.819044301375961 0.43929751410856177 0.5899983465325186; visual box size=0.819044301375961 0.43929751410856177 0.5899983465325186
- added link Link4, mass 1; collision box size=0.8164731214851686 0.3520826250216147 0.8781031911749925; visual box size=0.8164731214851686 0.3520826250216147 0.8781031911749925
- added link Link4Link50, mass 1; collision box size=0 0 0; visual box size=0 0 0
- added link Link4Link51, mass 1; collision box size=0 0 0; visual box size=0 0 0
- added link Link5, mass 1; collision box size=0.10934718806509791 0.8183067390840827 0.20280720384563444; visual box size=0.10934718806509791 0.8183067390840827 0.20280720384563444
- added link Link6, mass 1; collision box size=0.1623652540022137 0.1286602790825121 0.13057682767713918; visual box size=0.1623652540022137 0.1286602790825121 0.13057682767713918
- added link Link6Link70, mass 1; collision box size=0 0 0; visual box size=0 0 0
- added link Link6Link71, mass 1; collision box size=0 0 0; visual box size=0 0 0
- added link Link7, mass 1; collision box size=0.701495469889678 0.47348141229659524 0.043615791580008834; visual box size=0.701495469889678 0.47348141229659524 0.043615791580008834
- added link Link8, mass 1; collision box size=0.8053457493802818 0.031922397420427906 0.766896021226359; visual box size=0.8053457493802818 0.031922397420427906 0.766896021226359
- added link Link8Link90, mass 1; collision box size=0 0 0; visual box size=0 0 0
- added link Link8Link91, mass 1; collision box size=0 0 0; visual box size=0 0 0
- added link Link9, mass 1; collision box size=0.7500041573615707 0.025588693549430164 0.039846456288474275; visual box size=0.7500041573615707 0.025588693549430164 0.039846456288474275
- added link Link9Link100, mass 1; collision box size=0 0 0; visual box size=0 0 0
- link Link0: geometry collision box size=0.2676179393085856 0.053139138707052 0.8775790248727129; visual box size=0.2676179393085856 0.053139138707052 0.8775790248727129
- link Link1: geometry collision box size=0.9848497641438927 0.7217049589130019 0.998464422441744; visual box size=0.9848497641438927 0.7217049589130019 0.998464422441744
Joints:
- removed joint Link0Link10_Link0Link11
- removed joint Link0Link11_Link1
- added joint Link0Link10_Link1: type revolute, parent Link0Link10, child Link1, origin xyz=0 0 0 rpy=0 0 0, axis 0 1 0, limit lower=-3.14159 upper=3.14159 effort=0.0 velocity=0.0
- added joint Link10Link110_Link11: type revolute, parent Link10Link110, child Link11, origin xyz=0 0 0 rpy=0 0 0, axis 0 1 0, limit lower=-3.14159 upper=3.14159 effort=0.0 velocity=0.0
- added joint Link10_Link10Link110: type revolute, parent Link10, child Link10Link110, origin xyz=0 0.3440572245439849 0 rpy=0 0 0, axis 1 0 0, limit lower=-3.14159 upper=3.14159 effort=0.0 velocity=0.0
- added joint Link11Link120_Link12: type revolute, parent Link11Link120, child Link12, origin xyz=0 0 0 rpy=0 0 0, axis 0 1 0, limit lower=-3.14159 upper=3.14159 effort=0.0 velocity=0.0
- added joint Link11_Link11Link120: type revolute, parent Link11, child Link11Link120, origin xyz=0 0.7230499624108918 0 rpy=0 0 0, axis 1 0 0, limit lower=-3.14159 upper=3.14159 effort=0.0 velocity=0.0
- added joint Link12Link130_Link12Link131: type revolute, parent Link12Link130, child Link12Link131, origin xyz=0 0 0 rpy=0 0 0, axis 0 1 0, limit lower=-3.14159 upper=3.14159 effort=0.0 velocity=0.0
- added joint Link12Link131_Link13: type revolute, parent Link12Link131, child Link13, origin xyz=0 0 0 rpy=0 0 0, axis 0 0 1, limit lower=-3.14159 upper=3.14159 effort=0.0 velocity=0.0
- added joint Link12_Link12Link130: type revolute, parent Link12, child Link12Link130, origin xyz=0 0.5030481387881167 0 rpy=0 0 0, axis 1 0 0, limit lower=-3.14159 upper=3.14159 effort=0.0 velocity=0.0
- added joint Link13Link140_Link14: type revolute, parent Link13Link140, child Link14, origin xyz=0 0 0 rpy=0 0 0, axis 0 1 0, limit lower=-3.14159 upper=3.14159 effort=0.0 velocity=0.0
- added joint Link13_Link13Link140: type revolute, parent Link13, child Link13Link140, origin xyz=0 0.7066246726596259 0 rpy=0 0 0, axis 1 0 0, limit lower=-3.14159 upper=3.14159 effort=0.0 velocity=0.0
- added joint Link14Link150_Link14Link151: type revolute, parent Link14Link150, child Link14Link151, origin xyz=0 0 0 rpy=0 0 0, axis 1 0 0, limit lower=-3.14159 upper=3.14159 effort=0.0 velocity=0.0
- added joint Link14Link151_Link15: type revolute, parent Link14Link151, child Link15, origin xyz=0 0 0 rpy=0 0 0, axis 0 1 0, limit lower=-3.14159 upper=3.14159 effort=0.0 velocity=0.0
- added joint Link14_Link14Link150: type revolute, parent Link14, child Link14Link150, origin xyz=0 0.9429736253086106 0 rpy=0 0 0, axis 0 0 1, limit lower=-3.14159 upper=3.14159 effort=0.0 velocity=0.0
- added joint Link15_Link16: type revolute, parent Link15, child Link16, origin xyz=0 0.6057533568110886 0 rpy=0 0 0, axis 0 0 1, limit lower=-3.14159 upper=3.14159 effort=0.0 velocity=0.0
- added joint Link16Link170_Link16Link171: type revolute, parent Link16Link170, child Link16Link171, origin xyz=0 0 0 rpy=0 0 0, axis 0 0 1, limit lower=-3.14159 upper=3.14159 effort=0.0 velocity=0.0
- added joint Link16Link171_Link17: type revolute, parent Link16Link171, child Link17, origin xyz=0 0 0 rpy=0 0 0, axis 1 0 0, limit lower=-3.14159 upper=3.14159 effort=0.0 velocity=0.0
- added joint Link16_Link16Link170: type revolute, parent Link16, child Link16Link170, origin xyz=0 0.5518196335360861 0 rpy=0 0 0, axis 0 1 0, limit lower=-3.14159 upper=3.14159 effort=0.0 velocity=0.0
- added joint Link17Link180_Link17Link181: type revolute, parent Link17Link180, child Link17Link181, origin xyz=0 0 0 rpy=0 0 0, axis 0 1 0, limit lower=-3.14159 upper=3.14159 effort=0.0 velocity=0.0
- added joint Link17Link181_Link18: type revolute, parent Link17Link181, child Link18, origin xyz=0 0 0 rpy=0 0 0, axis 1 0 0, limit lower=-3.14159 upper=3.14159 effort=0.0 velocity=0.0
- added joint Link17_Link17Link180: type revolute, parent Link17, child Link17Link180, origin xyz=0 0.3840055679952633 0 rpy=0 0 0, axis 0 0 1, limit lower=-3.14159 upper=3.14159 effort=0.0 velocity=0.0
- added joint Link18Link190_Link18Link191: type revolute, parent Link18Link190, child Link18Link191, origin xyz=0 0 0 rpy=0 0 0, axis 0 1 0, limit lower=-3.14159 upper=3.14159 effort=0.0 velocity=0.0
- added joint Link18Link191_Link19: type revolute, parent Link18Link191, child Link19, origin xyz=0 0 0 rpy=0 0 0, axis 1 0 0, limit lower=-3.14159 upper=3.14159 effort=0.0 velocity=0.0
- added joint Link18_Link18Link190: type revolute, parent Link18, child Link18Link190, origin xyz=0 0.42962978375535 0 rpy=0 0 0, axis 0 0 1, limit lower=-3.14159 upper=3.14159 effort=0.0 velocity=0.0
- added joint Link1Link20_Link1Link21: type revolute, parent Link1Link20, child Link1Link21, origin xyz=0 0 0 rpy=0 0 0, axis 1 0 0, limit lower=-3.14159 upper=3.14159 effort=0.0 velocity=0.0
- added joint Link1Link21_Link2: type revolute, parent Link1Link21, child Link2, origin xyz=0 0 0 rpy=0 0 0, axis 0 0 1, limit lower=-3.14159 upper=3.14159 effort=0.0 velocity=0.0
- added joint Link1_Link1Link20: type revolute, parent Link1, child Link1Link20, origin xyz=0 0.7217049589130019 0 rpy=0 0 0, axis 0 1 0, limit lower=-3.14159 upper=3.14159 effort=0.0 velocity=0.0
- added joint Link2Link30_Link3: type revolute, parent Link2Link30, child Link3, origin xyz=0 0 0 rpy=0 0 0, axis 0 1 0, limit lower=-3.14159 upper=3.14159 effort=0.0 velocity=0.0
- added joint Link2_Link2Link30: type revolute, parent Link2, child Link2Link30, origin xyz=0 0.23912236519631302 0 rpy=0 0 0, axis 0 0 1, limit lower=-3.14159 upper=3.14159 effort=0.0 velocity=0.0
- added joint Link3_Link4: type revolute, parent Link3, child Link4, origin xyz=0 0.43929751410856177 0 rpy=0 0 0, axis 0 0 1, limit lower=-3.14159 upper=3.14159 effort=0.0 velocity=0.0
- added joint Link4Link50_Link4Link51: type revolute, parent Link4Link50, child Link4Link51, origin xyz=0 0 0 rpy=0 0 0, axis 0 1 0, limit lower=-3.14159 upper=3.14159 effort=0.0 velocity=0.0
- added joint Link4Link51_Link5: type revolute, parent Link4Link51, child Link5, origin xyz=0 0 0 rpy=0 0 0, axis 0 0 1, limit lower=-3.14159 upper=3.14159 effort=0.0 velocity=0.0
- added joint Link4_Link4Link50: type revolute, parent Link4, child Link4Link50, origin xyz=0 0.3520826250216147 0 rpy=0 0 0, axis 1 0 0, limit lower=-3.14159 upper=3.14159 effort=0.0 velocity=0.0
- added joint Link5_Link6: type revolute, parent Link5, child Link6, origin xyz=0 0.8183067390840827 0 rpy=0 0 0, axis 0 0 1, limit lower=-3.14159 upper=3.14159 effort=0.0 velocity=0.0
- added joint Link6Link70_Link6Link71: type revolute, parent Link6Link70, child Link6Link71, origin xyz=0 0 0 rpy=0 0 0, axis 0 0 1, limit lower=-3.14159 upper=3.14159 effort=0.0 velocity=0.0
- added joint Link6Link71_Link7: type revolute, parent Link6Link71, child Link7, origin xyz=0 0 0 rpy=0 0 0, axis 1 0 0, limit lower=-3.14159 upper=3.14159 effort=0.0 velocity=0.0
- added joint Link6_Link6Link70: type revolute, parent Link6, child Link6Link70, origin xyz=0 0.1286602790825121 0 rpy=0 0 0, axis 0 1 0, limit lower=-3.14159 upper=3.14159 effort=0.0 velocity=0.0
- added joint Link7_Link8: type revolute, parent Link7, child Link8, origin xyz=0 0.47348141229659524 0 rpy=0 0 0, axis 0 0 1, limit lower=-3.14159 upper=3.14159 effort=0.0 velocity=0.0
- added joint Link8Link90_Link8Link91: type revolute, parent Link8Link90, child Link8Link91, origin xyz=0 0 0 rpy=0 0 0, axis 1 0 0, limit lower=-3.14159 upper=3.14159 effort=0.0 velocity=0.0
- added joint Link8Link91_Link9: type revolute, parent Link8Link91, child Link9, origin xyz=0 0 0 rpy=0 0 0, axis 0 1 0, limit lower=-3.14159 upper=3.14159 effort=0.0 velocity=0.0
- added joint Link8_Link8Link90: type revolute, parent Link8, child Link8Link90, origin xyz=0 0.031922397420427906 0 rpy=0 0 0, axis 0 0 1, limit lower=-3.14159 upper=3.14159 effort=0.0 velocity=0.0
- added joint Link9Link100_Link10: type revolute, parent Link9Link100, child Link10, origin xyz=0 0 0 rpy=0 0 0, axis 0 0 1, limit lower=-3.14159 upper=3.14159 effort=0.0 velocity=0.0
- added joint Link9_Link9Link100: type revolute, parent Link9, child Link9Link100, origin xyz=0 0.025588693549430164 0 rpy=0 0 0, axis 1 0 0, limit lower=-3.14159 upper=3.14159 effort=0.0 velocity=0.0
- joint Link0_Link0Link10: axis 0 1 0 -> 1 0 0; origin xyz=0 0.2576103080702461 0.3288519841295286 rpy=0 0 0 -> xyz=0 0.026569569353526 0.499232211220872 rpy=0 0 0
