Commit message: cleanup

File: body.urdf (robot description, URDF)
Before this commit: robot robot, 44 links, 43 joints
Links:
- removed link Link10Link110
- removed link Link12Link130
- removed link Link12Link131
- removed link Link14Link150
- removed link Link14Link151
- removed link Link1Link21
- removed link Link6Link71
- removed link Link8Link91
- removed link Link9Link100
- added link Link11Link121, mass 1; collision box size=0 0 0; visual box size=0 0 0
- added link Link15Link160, mass 1; collision box size=0 0 0; visual box size=0 0 0
- added link Link15Link161, mass 1; collision box size=0 0 0; visual box size=0 0 0
- added link Link20, mass 1; collision box size=0.04435703097702992 0.9485163124606769 0.919430652917973; visual box size=0.04435703097702992 0.9485163124606769 0.919430652917973
- added link Link20Link210, mass 1; collision box size=0 0 0; visual box size=0 0 0
- added link Link20Link211, mass 1; collision box size=0 0 0; visual box size=0 0 0
- added link Link21, mass 1; collision box size=0.7500354627186304 0.08270097405336008 0.13591536297628415; visual box size=0.7500354627186304 0.08270097405336008 0.13591536297628415
- added link Link21Link220, mass 1; collision box size=0 0 0; visual box size=0 0 0
- added link Link21Link221, mass 1; collision box size=0 0 0; visual box size=0 0 0
- added link Link22, mass 1; collision box size=0.6020087663388213 0.8076388814142509 0.5547088738759718; visual box size=0.6020087663388213 0.8076388814142509 0.5547088738759718
- added link Link22Link230, mass 1; collision box size=0 0 0; visual box size=0 0 0
- added link Link23, mass 1; collision box size=0.06634654409195728 0.11579786840583373 0.5450216196625955; visual box size=0.06634654409195728 0.11579786840583373 0.5450216196625955
- added link Link24, mass 1; collision box size=0.33504294270204127 0.2743108056480392 0.3960269004930188; visual box size=0.33504294270204127 0.2743108056480392 0.3960269004930188
- added link Link25, mass 1; collision box size=0.26295257988737775 0.08353310708904949 0.9877128245614921; visual box size=0.26295257988737775 0.08353310708904949 0.9877128245614921
- added link Link25Link260, mass 1; collision box size=0 0 0; visual box size=0 0 0
- added link Link26, mass 1; collision box size=0.9870395777463543 0.3747798098193813 0.10452113603456459; visual box size=0.9870395777463543 0.3747798098193813 0.10452113603456459
- added link Link26Link270, mass 1; collision box size=0 0 0; visual box size=0 0 0
- added link Link27, mass 1; collision box size=0.11036745831044315 0.5735568451320422 0.388091537353341; visual box size=0.11036745831044315 0.5735568451320422 0.388091537353341
- added link Link27Link280, mass 1; collision box size=0 0 0; visual box size=0 0 0
- added link Link27Link281, mass 1; collision box size=0 0 0; visual box size=0 0 0
- added link Link28, mass 1; collision box size=0.12471707855637915 0.5025069915651947 0.03060887640011778; visual box size=0.12471707855637915 0.5025069915651947 0.03060887640011778
- added link Link28Link290, mass 1; collision box size=0 0 0; visual box size=0 0 0
- added link Link29, mass 1; collision box size=0.4803456297270339 0.8134882283486716 0.9202994244406573; visual box size=0.4803456297270339 0.8134882283486716 0.9202994244406573
- added link Link29Link300, mass 1; collision box size=0 0 0; visual box size=0 0 0
- added link Link30, mass 1; collision box size=0.9894238169582263 0.6414952987275251 0.5210769659476878; visual box size=0.9894238169582263 0.6414952987275251 0.5210769659476878
- added link Link30Link310, mass 1; collision box size=0 0 0; visual box size=0 0 0
- added link Link31, mass 1; collision box size=0.5756541278157986 0.4654098052991662 0.5074171772014103; visual box size=0.5756541278157986 0.4654098052991662 0.5074171772014103
- added link Link31Link320, mass 1; collision box size=0 0 0; visual box size=0 0 0
- added link Link32, mass 1; collision box size=0.873112028611666 0.010295739544902593 0.792089102849323; visual box size=0.873112028611666 0.010295739544902593 0.792089102849323
- added link Link32Link330, mass 1; collision box size=0 0 0; visual box size=0 0 0
- added link Link32Link331, mass 1; collision box size=0 0 0; visual box size=0 0 0
- added link Link33, mass 1; collision box size=0.2319924785954497 0.03955845925894996 0.5639679140144899; visual box size=0.2319924785954497 0.03955845925894996 0.5639679140144899
- added link Link34, mass 1; collision box size=0.9736716366954478 0.7902099723813645 0.15373806578654847; visual box size=0.9736716366954478 0.7902099723813645 0.15373806578654847
- added link Link34Link350, mass 1; collision box size=0 0 0; visual box size=0 0 0
- added link Link35, mass 1; collision box size=0.8706871190062832 0.9729056220236582 0.3082847792952471; visual box size=0.8706871190062832 0.9729056220236582 0.3082847792952471
- added link Link36, mass 1; collision box size=0.836025200019191 0.12403379509665757 0.5344252186706308; visual box size=0.836025200019191 0.12403379509665757 0.5344252186706308
- added link Link37, mass 1; collision box size=0.6518816351968165 0.12654397306599752 0.8155165643574079; visual box size=0.6518816351968165 0.12654397306599752 0.8155165643574079
- added link Link37Link380, mass 1; collision box size=0 0 0; visual box size=0 0 0
- added link Link37Link381, mass 1; collision box size=0 0 0; visual box size=0 0 0
- added link Link38, mass 1; collision box size=0.6368779883991167 0.2764907663190408 0.6229438808461755; visual box size=0.6368779883991167 0.2764907663190408 0.6229438808461755
- added link Link38Link390, mass 1; collision box size=0 0 0; visual box size=0 0 0
- added link Link39, mass 1; collision box size=0.4430962027290417 0.6196858110549571 0.3942365424887705; visual box size=0.4430962027290417 0.6196858110549571 0.3942365424887705
- added link Link39Link400, mass 1; collision box size=0 0 0; visual box size=0 0 0
- added link Link40, mass 1; collision box size=0.467086216954649 0.28528844984068513 0.737182793156155; visual box size=0.467086216954649 0.28528844984068513 0.737182793156155
- added link Link40Link410, mass 1; collision box size=0 0 0; visual box size=0 0 0
- added link Link40Link411, mass 1; collision box size=0 0 0; visual box size=0 0 0
- added link Link41, mass 1; collision box size=0.1953630178644311 0.6360824021694144 0.29569237671845605; visual box size=0.1953630178644311 0.6360824021694144 0.29569237671845605
- added link Link41Link420, mass 1; collision box size=0 0 0; visual box size=0 0 0
- added link Link42, mass 1; collision box size=0.024797240922265762 0.05334507668755384 0.295105893957171; visual box size=0.024797240922265762 0.05334507668755384 0.295105893957171
- added link Link43, mass 1; collision box size=0.14253248173813726 0.33887107177902775 0.9590531691002383; visual box size=0.14253248173813726 0.33887107177902775 0.9590531691002383
- added link Link43Link440, mass 1; collision box size=0 0 0; visual box size=0 0 0
- added link Link43Link441, mass 1; collision box size=0 0 0; visual box size=0 0 0
- added link Link44, mass 1; collision box size=0.6902614870080568 0.8839166090238865 0.027706394356107222; visual box size=0.6902614870080568 0.8839166090238865 0.027706394356107222
- added link Link45, mass 1; collision box size=0.732319685746325 0.6912042219257425 0.4030567887441737; visual box size=0.732319685746325 0.6912042219257425 0.4030567887441737
- added link Link45Link460, mass 1; collision box size=0 0 0; visual box size=0 0 0
- added link Link45Link461, mass 1; collision box size=0 0 0; visual box size=0 0 0
- added link Link46, mass 1; collision box size=0.6880929931469454 0.20631636945401288 0.6735883391017942; visual box size=0.6880929931469454 0.20631636945401288 0.6735883391017942
- added link Link46Link470, mass 1; collision box size=0 0 0; visual box size=0 0 0
- added link Link46Link471, mass 1; collision box size=0 0 0; visual box size=0 0 0
- added link Link47, mass 1; collision box size=0.5248028351900028 0.971475420319286 0.8025922122057157; visual box size=0.5248028351900028 0.971475420319286 0.8025922122057157
- added link Link48, mass 1; collision box size=0.44465258052928025 0.21640484362919354 0.4422539953498237; visual box size=0.44465258052928025 0.21640484362919354 0.4422539953498237
- added link Link48Link490, mass 1; collision box size=0 0 0; visual box size=0 0 0
- added link Link49, mass 1; collision box size=0.9541298997077117 0.05029545638251731 0.6841322924839255; visual box size=0.9541298997077117 0.05029545638251731 0.6841322924839255
- added link Link7Link80, mass 1; collision box size=0 0 0; visual box size=0 0 0
- added link Link7Link81, mass 1; collision box size=0 0 0; visual box size=0 0 0
- link Link0: geometry collision box size=0.9286088413248901 0.22375245541877853 0.37524030187148005; visual box size=0.9286088413248901 0.22375245541877853 0.37524030187148005
- link Link1: geometry collision box size=0.662037003478744 0.18593653607767813 0.970399417640562; visual box size=0.662037003478744 0.18593653607767813 0.970399417640562
- link Link10: geometry collision box size=0.2735609775678307 0.19616040873250717 0.03785319934779374; visual box size=0.2735609775678307 0.19616040873250717 0.03785319934779374
- link Link11: geometry collision box size=0.20145731105180298 0.11194042901805223 0.26872172088513147; visual box size=0.20145731105180298 0.11194042901805223 0.26872172088513147
- link Link12: geometry collision box size=0.6216308322646081 0.34618948282382556 0.1158699936661659; visual box size=0.6216308322646081 0.34618948282382556 0.1158699936661659
- link Link13: geometry collision box size=0.04844989826873036 0.03163308527476549 0.6001294921682481; visual box size=0.04844989826873036 0.03163308527476549 0.6001294921682481
- link Link14: geometry collision box size=0.934709521815948 0.990197465945178 0.9821962436450067; visual box size=0.934709521815948 0.990197465945178 0.9821962436450067
- link Link15: geometry collision box size=0.2864895896258216 0.11846191806246065 0.9877089415578786; visual box size=0.2864895896258216 0.11846191806246065 0.9877089415578786
- link Link16: geometry collision box size=0.2602883691825907 0.8720986046159597 0.4137331848995911; visual box size=0.2602883691825907 0.8720986046159597 0.4137331848995911
- link Link17: geometry collision box size=0.19997354955104651 0.5416733857509541 0.10341024147373201; visual box size=0.19997354955104651 0.5416733857509541 0.10341024147373201
- link Link18: geometry collision box size=0.38146215482384593 0.9405170045343042 0.06458045113338151; visual box size=0.38146215482384593 0.9405170045343042 0.06458045113338151
- link Link19: geometry collision box size=0.03905446735530094 0.5667023006758852 0.06714949390338121; visual box size=0.03905446735530094 0.5667023006758852 0.06714949390338121
- link Link2: geometry collision box size=0.09221926226896138 0.982230039474184 0.039201498369309085; visual box size=0.09221926226896138 0.982230039474184 0.039201498369309085
- link Link3: geometry collision box size=0.9229437327328965 0.04937157675223747 0.5259393381864983; visual box size=0.9229437327328965 0.04937157675223747 0.5259393381864983
- link Link4: geometry collision box size=0.37906394519302566 0.33510369557687447 0.21314168687853652; visual box size=0.37906394519302566 0.33510369557687447 0.21314168687853652
- link Link5: geometry collision box size=0.1540127097272158 0.29378298482862486 0.7212493325237628; visual box size=0.1540127097272158 0.29378298482862486 0.7212493325237628
- link Link6: geometry collision box size=0.8911318765952263 0.9465924498551117 0.46176104004774954; visual box size=0.8911318765952263 0.9465924498551117 0.46176104004774954
- link Link7: geometry collision box size=0.5677213684809213 0.9496152988545844 0.5063839841280126; visual box size=0.5677213684809213 0.9496152988545844 0.5063839841280126
- link Link8: geometry collision box size=0.5254078537130686 0.7232970218814561 0.7839101928797775; visual box size=0.5254078537130686 0.7232970218814561 0.7839101928797775
- link Link9: geometry collision box size=0.2555960367347393 0.28098950319604443 0.8457992554410558; visual box size=0.2555960367347393 0.28098950319604443 0.8457992554410558
Joints:
- removed joint Link10Link110_Link11
- removed joint Link10_Link10Link110
- removed joint Link11Link120_Link12
- removed joint Link12Link130_Link12Link131
- removed joint Link12Link131_Link13
- removed joint Link12_Link12Link130
- removed joint Link14Link150_Link14Link151
- removed joint Link14Link151_Link15
- removed joint Link14_Link14Link150
- removed joint Link15_Link16
- removed joint Link1Link20_Link1Link21
- removed joint Link1Link21_Link2
- removed joint Link6Link70_Link6Link71
- removed joint Link6Link71_Link7
- removed joint Link7_Link8
- removed joint Link8Link90_Link8Link91
- removed joint Link8Link91_Link9
- removed joint Link9Link100_Link10
- removed joint Link9_Link9Link100
- added joint Link10_Link11: type revolute, parent Link10, child Link11, origin xyz=0 0.19616040873250717 0 rpy=0 0 0, axis 1 0 0, limit lower=-3.14159 upper=3.14159 effort=0.0 velocity=0.0
- added joint Link11Link120_Link11Link121: type revolute, parent Link11Link120, child Link11Link121, origin xyz=0 0 0 rpy=0 0 0, axis 0 0 1, limit lower=-3.14159 upper=3.14159 effort=0.0 velocity=0.0
- added joint Link11Link121_Link12: type revolute, parent Link11Link121, child Link12, origin xyz=0 0 0 rpy=0 0 0, axis 1 0 0, limit lower=-3.14159 upper=3.14159 effort=0.0 velocity=0.0
- added joint Link12_Link13: type revolute, parent Link12, child Link13, origin xyz=0 0.34618948282382556 0 rpy=0 0 0, axis 0 0 1, limit lower=-3.14159 upper=3.14159 effort=0.0 velocity=0.0
- added joint Link14_Link15: type revolute, parent Link14, child Link15, origin xyz=0 0.990197465945178 0 rpy=0 0 0, axis 1 0 0, limit lower=-3.14159 upper=3.14159 effort=0.0 velocity=0.0
- added joint Link15Link160_Link15Link161: type revolute, parent Link15Link160, child Link15Link161, origin xyz=0 0 0 rpy=0 0 0, axis 1 0 0, limit lower=-3.14159 upper=3.14159 effort=0.0 velocity=0.0
- added joint Link15Link161_Link16: type revolute, parent Link15Link161, child Link16, origin xyz=0 0 0 rpy=0 0 0, axis 0 0 1, limit lower=-3.14159 upper=3.14159 effort=0.0 velocity=0.0
- added joint Link15_Link15Link160: type revolute, parent Link15, child Link15Link160, origin xyz=0 0.11846191806246065 0 rpy=0 0 0, axis 0 1 0, limit lower=-3.14159 upper=3.14159 effort=0.0 velocity=0.0
- added joint Link19_Link20: type revolute, parent Link19, child Link20, origin xyz=0 0.5667023006758852 0 rpy=0 0 0, axis 1 0 0, limit lower=-3.14159 upper=3.14159 effort=0.0 velocity=0.0
- added joint Link1Link20_Link2: type revolute, parent Link1Link20, child Link2, origin xyz=0 0 0 rpy=0 0 0, axis 0 0 1, limit lower=-3.14159 upper=3.14159 effort=0.0 velocity=0.0
- added joint Link20Link210_Link20Link211: type revolute, parent Link20Link210, child Link20Link211, origin xyz=0 0 0 rpy=0 0 0, axis 0 0 1, limit lower=-3.14159 upper=3.14159 effort=0.0 velocity=0.0
- added joint Link20Link211_Link21: type revolute, parent Link20Link211, child Link21, origin xyz=0 0 0 rpy=0 0 0, axis 1 0 0, limit lower=-3.14159 upper=3.14159 effort=0.0 velocity=0.0
- added joint Link20_Link20Link210: type revolute, parent Link20, child Link20Link210, origin xyz=0 0.9485163124606769 0 rpy=0 0 0, axis 0 1 0, limit lower=-3.14159 upper=3.14159 effort=0.0 velocity=0.0
- added joint Link21Link220_Link21Link221: type revolute, parent Link21Link220, child Link21Link221, origin xyz=0 0 0 rpy=0 0 0, axis 0 1 0, limit lower=-3.14159 upper=3.14159 effort=0.0 velocity=0.0
- added joint Link21Link221_Link22: type revolute, parent Link21Link221, child Link22, origin xyz=0 0 0 rpy=0 0 0, axis 1 0 0, limit lower=-3.14159 upper=3.14159 effort=0.0 velocity=0.0
- added joint Link21_Link21Link220: type revolute, parent Link21, child Link21Link220, origin xyz=0 0.08270097405336008 0 rpy=0 0 0, axis 0 0 1, limit lower=-3.14159 upper=3.14159 effort=0.0 velocity=0.0
- added joint Link22Link230_Link23: type revolute, parent Link22Link230, child Link23, origin xyz=0 0 0 rpy=0 0 0, axis 1 0 0, limit lower=-3.14159 upper=3.14159 effort=0.0 velocity=0.0
- added joint Link22_Link22Link230: type revolute, parent Link22, child Link22Link230, origin xyz=0 0.8076388814142509 0 rpy=0 0 0, axis 0 1 0, limit lower=-3.14159 upper=3.14159 effort=0.0 velocity=0.0
- added joint Link23_Link24: type revolute, parent Link23, child Link24, origin xyz=0 0.11579786840583373 0 rpy=0 0 0, axis 0 1 0, limit lower=-3.14159 upper=3.14159 effort=0.0 velocity=0.0
- added joint Link24_Link25: type revolute, parent Link24, child Link25, origin xyz=0 0.2743108056480392 0 rpy=0 0 0, axis 1 0 0, limit lower=-3.14159 upper=3.14159 effort=0.0 velocity=0.0
- added joint Link25Link260_Link26: type revolute, parent Link25Link260, child Link26, origin xyz=0 0 0 rpy=0 0 0, axis 0 1 0, limit lower=-3.14159 upper=3.14159 effort=0.0 velocity=0.0
- added joint Link25_Link25Link260: type revolute, parent Link25, child Link25Link260, origin xyz=0 0.08353310708904949 0 rpy=0 0 0, axis 0 0 1, limit lower=-3.14159 upper=3.14159 effort=0.0 velocity=0.0
- added joint Link26Link270_Link27: type revolute, parent Link26Link270, child Link27, origin xyz=0 0 0 rpy=0 0 0, axis 0 1 0, limit lower=-3.14159 upper=3.14159 effort=0.0 velocity=0.0
- added joint Link26_Link26Link270: type revolute, parent Link26, child Link26Link270, origin xyz=0 0.3747798098193813 0 rpy=0 0 0, axis 0 0 1, limit lower=-3.14159 upper=3.14159 effort=0.0 velocity=0.0
- added joint Link27Link280_Link27Link281: type revolute, parent Link27Link280, child Link27Link281, origin xyz=0 0 0 rpy=0 0 0, axis 0 1 0, limit lower=-3.14159 upper=3.14159 effort=0.0 velocity=0.0
- added joint Link27Link281_Link28: type revolute, parent Link27Link281, child Link28, origin xyz=0 0 0 rpy=0 0 0, axis 0 0 1, limit lower=-3.14159 upper=3.14159 effort=0.0 velocity=0.0
- added joint Link27_Link27Link280: type revolute, parent Link27, child Link27Link280, origin xyz=0 0.5735568451320422 0 rpy=0 0 0, axis 1 0 0, limit lower=-3.14159 upper=3.14159 effort=0.0 velocity=0.0
- added joint Link28Link290_Link29: type revolute, parent Link28Link290, child Link29, origin xyz=0 0 0 rpy=0 0 0, axis 0 1 0, limit lower=-3.14159 upper=3.14159 effort=0.0 velocity=0.0
- added joint Link28_Link28Link290: type revolute, parent Link28, child Link28Link290, origin xyz=0 0.5025069915651947 0 rpy=0 0 0, axis 1 0 0, limit lower=-3.14159 upper=3.14159 effort=0.0 velocity=0.0
- added joint Link29Link300_Link30: type revolute, parent Link29Link300, child Link30, origin xyz=0 0 0 rpy=0 0 0, axis 1 0 0, limit lower=-3.14159 upper=3.14159 effort=0.0 velocity=0.0
- added joint Link29_Link29Link300: type revolute, parent Link29, child Link29Link300, origin xyz=0 0.8134882283486716 0 rpy=0 0 0, axis 0 1 0, limit lower=-3.14159 upper=3.14159 effort=0.0 velocity=0.0
- added joint Link30Link310_Link31: type revolute, parent Link30Link310, child Link31, origin xyz=0 0 0 rpy=0 0 0, axis 0 0 1, limit lower=-3.14159 upper=3.14159 effort=0.0 velocity=0.0
- added joint Link30_Link30Link310: type revolute, parent Link30, child Link30Link310, origin xyz=0 0.6414952987275251 0 rpy=0 0 0, axis 1 0 0, limit lower=-3.14159 upper=3.14159 effort=0.0 velocity=0.0
- added joint Link31Link320_Link32: type revolute, parent Link31Link320, child Link32, origin xyz=0 0 0 rpy=0 0 0, axis 0 0 1, limit lower=-3.14159 upper=3.14159 effort=0.0 velocity=0.0
- added joint Link31_Link31Link320: type revolute, parent Link31, child Link31Link320, origin xyz=0 0.4654098052991662 0 rpy=0 0 0, axis 0 1 0, limit lower=-3.14159 upper=3.14159 effort=0.0 velocity=0.0
- added joint Link32Link330_Link32Link331: type revolute, parent Link32Link330, child Link32Link331, origin xyz=0 0 0 rpy=0 0 0, axis 0 1 0, limit lower=-3.14159 upper=3.14159 effort=0.0 velocity=0.0
- added joint Link32Link331_Link33: type revolute, parent Link32Link331, child Link33, origin xyz=0 0 0 rpy=0 0 0, axis 1 0 0, limit lower=-3.14159 upper=3.14159 effort=0.0 velocity=0.0
- added joint Link32_Link32Link330: type revolute, parent Link32, child Link32Link330, origin xyz=0 0.010295739544902593 0 rpy=0 0 0, axis 0 0 1, limit lower=-3.14159 upper=3.14159 effort=0.0 velocity=0.0
- added joint Link33_Link34: type revolute, parent Link33, child Link34, origin xyz=0 0.03955845925894996 0 rpy=0 0 0, axis 1 0 0, limit lower=-3.14159 upper=3.14159 effort=0.0 velocity=0.0
- added joint Link34Link350_Link35: type revolute, parent Link34Link350, child Link35, origin xyz=0 0 0 rpy=0 0 0, axis 1 0 0, limit lower=-3.14159 upper=3.14159 effort=0.0 velocity=0.0
- added joint Link34_Link34Link350: type revolute, parent Link34, child Link34Link350, origin xyz=0 0.7902099723813645 0 rpy=0 0 0, axis 0 0 1, limit lower=-3.14159 upper=3.14159 effort=0.0 velocity=0.0
- added joint Link35_Link36: type revolute, parent Link35, child Link36, origin xyz=0 0.9729056220236582 0 rpy=0 0 0, axis 0 0 1, limit lower=-3.14159 upper=3.14159 effort=0.0 velocity=0.0
- added joint Link36_Link37: type revolute, parent Link36, child Link37, origin xyz=0 0.12403379509665757 0 rpy=0 0 0, axis 0 0 1, limit lower=-3.14159 upper=3.14159 effort=0.0 velocity=0.0
- added joint Link37Link380_Link37Link381: type revolute, parent Link37Link380, child Link37Link381, origin xyz=0 0 0 rpy=0 0 0, axis 0 1 0, limit lower=-3.14159 upper=3.14159 effort=0.0 velocity=0.0
- added joint Link37Link381_Link38: type revolute, parent Link37Link381, child Link38, origin xyz=0 0 0 rpy=0 0 0, axis 0 0 1, limit lower=-3.14159 upper=3.14159 effort=0.0 velocity=0.0
- added joint Link37_Link37Link380: type revolute, parent Link37, child Link37Link380, origin xyz=0 0.12654397306599752 0 rpy=0 0 0, axis 1 0 0, limit lower=-3.14159 upper=3.14159 effort=0.0 velocity=0.0
- added joint Link38Link390_Link39: type revolute, parent Link38Link390, child Link39, origin xyz=0 0 0 rpy=0 0 0, axis 0 1 0, limit lower=-3.14159 upper=3.14159 effort=0.0 velocity=0.0
- added joint Link38_Link38Link390: type revolute, parent Link38, child Link38Link390, origin xyz=0 0.2764907663190408 0 rpy=0 0 0, axis 1 0 0, limit lower=-3.14159 upper=3.14159 effort=0.0 velocity=0.0
- added joint Link39Link400_Link40: type revolute, parent Link39Link400, child Link40, origin xyz=0 0 0 rpy=0 0 0, axis 0 1 0, limit lower=-3.14159 upper=3.14159 effort=0.0 velocity=0.0
- added joint Link39_Link39Link400: type revolute, parent Link39, child Link39Link400, origin xyz=0 0.6196858110549571 0 rpy=0 0 0, axis 1 0 0, limit lower=-3.14159 upper=3.14159 effort=0.0 velocity=0.0
- added joint Link40Link410_Link40Link411: type revolute, parent Link40Link410, child Link40Link411, origin xyz=0 0 0 rpy=0 0 0, axis 0 0 1, limit lower=-3.14159 upper=3.14159 effort=0.0 velocity=0.0
- added joint Link40Link411_Link41: type revolute, parent Link40Link411, child Link41, origin xyz=0 0 0 rpy=0 0 0, axis 1 0 0, limit lower=-3.14159 upper=3.14159 effort=0.0 velocity=0.0
- added joint Link40_Link40Link410: type revolute, parent Link40, child Link40Link410, origin xyz=0 0.28528844984068513 0 rpy=0 0 0, axis 0 1 0, limit lower=-3.14159 upper=3.14159 effort=0.0 velocity=0.0
- added joint Link41Link420_Link42: type revolute, parent Link41Link420, child Link42, origin xyz=0 0 0 rpy=0 0 0, axis 1 0 0, limit lower=-3.14159 upper=3.14159 effort=0.0 velocity=0.0
- added joint Link41_Link41Link420: type revolute, parent Link41, child Link41Link420, origin xyz=0 0.6360824021694144 0 rpy=0 0 0, axis 0 0 1, limit lower=-3.14159 upper=3.14159 effort=0.0 velocity=0.0
- added joint Link42_Link43: type revolute, parent Link42, child Link43, origin xyz=0 0.05334507668755384 0 rpy=0 0 0, axis 0 1 0, limit lower=-3.14159 upper=3.14159 effort=0.0 velocity=0.0
- added joint Link43Link440_Link43Link441: type revolute, parent Link43Link440, child Link43Link441, origin xyz=0 0 0 rpy=0 0 0, axis 0 1 0, limit lower=-3.14159 upper=3.14159 effort=0.0 velocity=0.0
- added joint Link43Link441_Link44: type revolute, parent Link43Link441, child Link44, origin xyz=0 0 0 rpy=0 0 0, axis 1 0 0, limit lower=-3.14159 upper=3.14159 effort=0.0 velocity=0.0
- added joint Link43_Link43Link440: type revolute, parent Link43, child Link43Link440, origin xyz=0 0.33887107177902775 0 rpy=0 0 0, axis 0 0 1, limit lower=-3.14159 upper=3.14159 effort=0.0 velocity=0.0
- added joint Link44_Link45: type revolute, parent Link44, child Link45, origin xyz=0 0.8839166090238865 0 rpy=0 0 0, axis 0 1 0, limit lower=-3.14159 upper=3.14159 effort=0.0 velocity=0.0
- added joint Link45Link460_Link45Link461: type revolute, parent Link45Link460, child Link45Link461, origin xyz=0 0 0 rpy=0 0 0, axis 0 1 0, limit lower=-3.14159 upper=3.14159 effort=0.0 velocity=0.0
- added joint Link45Link461_Link46: type revolute, parent Link45Link461, child Link46, origin xyz=0 0 0 rpy=0 0 0, axis 1 0 0, limit lower=-3.14159 upper=3.14159 effort=0.0 velocity=0.0
- added joint Link45_Link45Link460: type revolute, parent Link45, child Link45Link460, origin xyz=0 0.6912042219257425 0 rpy=0 0 0, axis 0 0 1, limit lower=-3.14159 upper=3.14159 effort=0.0 velocity=0.0
- added joint Link46Link470_Link46Link471: type revolute, parent Link46Link470, child Link46Link471, origin xyz=0 0 0 rpy=0 0 0, axis 1 0 0, limit lower=-3.14159 upper=3.14159 effort=0.0 velocity=0.0
- added joint Link46Link471_Link47: type revolute, parent Link46Link471, child Link47, origin xyz=0 0 0 rpy=0 0 0, axis 0 0 1, limit lower=-3.14159 upper=3.14159 effort=0.0 velocity=0.0
- added joint Link46_Link46Link470: type revolute, parent Link46, child Link46Link470, origin xyz=0 0.20631636945401288 0 rpy=0 0 0, axis 0 1 0, limit lower=-3.14159 upper=3.14159 effort=0.0 velocity=0.0
- added joint Link47_Link48: type revolute, parent Link47, child Link48, origin xyz=0 0.971475420319286 0 rpy=0 0 0, axis 1 0 0, limit lower=-3.14159 upper=3.14159 effort=0.0 velocity=0.0
- added joint Link48Link490_Link49: type revolute, parent Link48Link490, child Link49, origin xyz=0 0 0 rpy=0 0 0, axis 0 1 0, limit lower=-3.14159 upper=3.14159 effort=0.0 velocity=0.0
- added joint Link48_Link48Link490: type revolute, parent Link48, child Link48Link490, origin xyz=0 0.21640484362919354 0 rpy=0 0 0, axis 1 0 0, limit lower=-3.14159 upper=3.14159 effort=0.0 velocity=0.0
- added joint Link6Link70_Link7: type revolute, parent Link6Link70, child Link7, origin xyz=0 0 0 rpy=0 0 0, axis 1 0 0, limit lower=-3.14159 upper=3.14159 effort=0.0 velocity=0.0
- added joint Link7Link80_Link7Link81: type revolute, parent Link7Link80, child Link7Link81, origin xyz=0 0 0 rpy=0 0 0, axis 1 0 0, limit lower=-3.14159 upper=3.14159 effort=0.0 velocity=0.0
- added joint Link7Link81_Link8: type revolute, parent Link7Link81, child Link8, origin xyz=0 0 0 rpy=0 0 0, axis 0 1 0, limit lower=-3.14159 upper=3.14159 effort=0.0 velocity=0.0
- added joint Link7_Link7Link80: type revolute, parent Link7, child Link7Link80, origin xyz=0 0.9496152988545844 0 rpy=0 0 0, axis 0 0 1, limit lower=-3.14159 upper=3.14159 effort=0.0 velocity=0.0
- added joint Link8Link90_Link9: type revolute, parent Link8Link90, child Link9, origin xyz=0 0 0 rpy=0 0 0, axis 0 0 1, limit lower=-3.14159 upper=3.14159 effort=0.0 velocity=0.0
- added joint Link9_Link10: type revolute, parent Link9, child Link10, origin xyz=0 0.28098950319604443 0 rpy=0 0 0, axis 0 1 0, limit lower=-3.14159 upper=3.14159 effort=0.0 velocity=0.0
- joint Link0Link10_Link1: axis 0 1 0 -> 0 0 1
- joint Link0_Link0Link10: origin xyz=0 0.026569569353526 0.499232211220872 rpy=0 0 0 -> xyz=0 0.11187622770938926 0.49385641228074606 rpy=0 0 0
- joint Link11_Link11Link120: axis 1 0 0 -> 0 1 0; origin xyz=0 0.7230499624108918 0 rpy=0 0 0 -> xyz=0 0.11194042901805223 0 rpy=0 0 0
- joint Link13Link140_Link14: axis 0 1 0 -> 1 0 0
- joint Link13_Link13Link140: axis 1 0 0 -> 0 1 0; origin xyz=0 0.7066246726596259 0 rpy=0 0 0 -> xyz=0 0.03163308527476549 0 rpy=0 0 0
- joint Link16Link170_Link16Link171: axis 0 0 1 -> 1 0 0
- joint Link16Link171_Link17: axis 1 0 0 -> 0 0 1
- joint Link16_Link16Link170: origin xyz=0 0.5518196335360861 0 rpy=0 0 0 -> xyz=0 0.8720986046159597 0 rpy=0 0 0
- joint Link17Link180_Link17Link181: axis 0 1 0 -> 1 0 0
- joint Link17Link181_Link18: axis 1 0 0 -> 0 0 1
- joint Link17_Link17Link180: axis 0 0 1 -> 0 1 0; origin xyz=0 0.3840055679952633 0 rpy=0 0 0 -> xyz=0 0.5416733857509541 0 rpy=0 0 0
- joint Link18Link190_Link18Link191: axis 0 1 0 -> 1 0 0
- joint Link18Link191_Link19: axis 1 0 0 -> 0 1 0
- joint Link18_Link18Link190: origin xyz=0 0.42962978375535 0 rpy=0 0 0 -> xyz=0 0.9405170045343042 0 rpy=0 0 0
- joint Link1_Link1Link20: axis 0 1 0 -> 1 0 0; origin xyz=0 0.7217049589130019 0 rpy=0 0 0 -> xyz=0 0.18593653607767813 0 rpy=0 0 0
- joint Link2Link30_Link3: axis 0 1 0 -> 1 0 0
- joint Link2_Link2Link30: origin xyz=0 0.23912236519631302 0 rpy=0 0 0 -> xyz=0 0.982230039474184 0 rpy=0 0 0
- joint Link3_Link4: axis 0 0 1 -> 0 1 0; origin xyz=0 0.43929751410856177 0 rpy=0 0 0 -> xyz=0 0.04937157675223747 0 rpy=0 0 0
- joint Link4Link50_Link4Link51: axis 0 1 0 -> 1 0 0
- joint Link4_Link4Link50: axis 1 0 0 -> 0 1 0; origin xyz=0 0.3520826250216147 0 rpy=0 0 0 -> xyz=0 0.33510369557687447 0 rpy=0 0 0
- joint Link5_Link6: axis 0 0 1 -> 0 1 0; origin xyz=0 0.8183067390840827 0 rpy=0 0 0 -> xyz=0 0.29378298482862486 0 rpy=0 0 0
- joint Link6_Link6Link70: axis 0 1 0 -> 0 0 1; origin xyz=0 0.1286602790825121 0 rpy=0 0 0 -> xyz=0 0.9465924498551117 0 rpy=0 0 0
- joint Link8_Link8Link90: axis 0 0 1 -> 0 1 0; origin xyz=0 0.031922397420427906 0 rpy=0 0 0 -> xyz=0 0.7232970218814561 0 rpy=0 0 0
