Commit message: 3d generation, no collision detection yet

File: body.urdf (robot description, URDF)
Before this commit: robot robot, 100 links, 99 joints
Links:
- removed link Link11Link120
- removed link Link11Link121
- removed link Link15
- removed link Link15Link160
- removed link Link15Link161
- removed link Link16
- removed link Link16Link170
- removed link Link16Link171
- removed link Link17
- removed link Link17Link180
- removed link Link17Link181
- removed link Link18
- removed link Link18Link190
- removed link Link18Link191
- removed link Link19
- removed link Link20
- removed link Link20Link210
- removed link Link20Link211
- removed link Link21
- removed link Link21Link220
- removed link Link21Link221
- removed link Link22
- removed link Link22Link230
- removed link Link23
- removed link Link24
- removed link Link25
- removed link Link25Link260
- removed link Link26
- removed link Link26Link270
- removed link Link27
- removed link Link27Link280
- removed link Link27Link281
- removed link Link28
- removed link Link28Link290
- removed link Link29
- removed link Link29Link300
- removed link Link2Link30
- removed link Link30
- removed link Link30Link310
- removed link Link31
- removed link Link31Link320
- removed link Link32
- removed link Link32Link330
- removed link Link32Link331
- removed link Link33
- removed link Link34
- removed link Link34Link350
- removed link Link35
- removed link Link36
- removed link Link37
- removed link Link37Link380
- removed link Link37Link381
- removed link Link38
- removed link Link38Link390
- removed link Link39
- removed link Link39Link400
- removed link Link40
- removed link Link40Link410
- removed link Link40Link411
- removed link Link41
- removed link Link41Link420
- removed link Link42
- removed link Link43
- removed link Link43Link440
- removed link Link43Link441
- removed link Link44
- removed link Link45
- removed link Link45Link460
- removed link Link45Link461
- removed link Link46
- removed link Link46Link470
- removed link Link46Link471
- removed link Link47
- removed link Link48
- removed link Link48Link490
- removed link Link49
- removed link Link4Link51
- removed link Link8Link90
- added link Link10Link110, mass 1; collision box size=0 0 0; visual box size=0 0 0
- added link Link13Link141, mass 1; collision box size=0 0 0; visual box size=0 0 0
- added link Link3Link40, mass 1; collision box size=0 0 0; visual box size=0 0 0
- added link Link5Link60, mass 1; collision box size=0 0 0; visual box size=0 0 0
- added link Link5Link61, mass 1; collision box size=0 0 0; visual box size=0 0 0
- added link Link6Link71, mass 1; collision box size=0 0 0; visual box size=0 0 0
- link Link0: geometry collision box size=0.5995758370939342 0.5919530484709288 0.2447891783915651; visual box size=0.5995758370939342 0.5919530484709288 0.2447891783915651
- link Link1: geometry collision box size=0.181960108546952 0.6996585355271348 0.43268059044153007; visual box size=0.181960108546952 0.6996585355271348 0.43268059044153007
- link Link10: geometry collision box size=0.22038294350318832 0.1543028465755263 0.6130190567397192; visual box size=0.22038294350318832 0.1543028465755263 0.6130190567397192
- link Link11: geometry collision box size=0.22545069783103056 0.7089102812992598 0.5116508421436593; visual box size=0.22545069783103056 0.7089102812992598 0.5116508421436593
- link Link12: geometry collision box size=0.16120087707033393 0.7239819482944811 0.22850724893198404; visual box size=0.16120087707033393 0.7239819482944811 0.22850724893198404
- link Link13: geometry collision box size=0.5818124517353301 0.20110454623322394 0.5866500676050811; visual box size=0.5818124517353301 0.20110454623322394 0.5866500676050811
- link Link14: geometry collision box size=0.544758212911489 0.385767501193494 0.8522107893250819; visual box size=0.544758212911489 0.385767501193494 0.8522107893250819
- link Link2: geometry collision box size=0.27406209550304383 0.8593048428928121 0.2605292615328091; visual box size=0.27406209550304383 0.8593048428928121 0.2605292615328091
- link Link3: geometry collision box size=0.059743190185429285 0.40109764424489613 0.8967900151447522; visual box size=0.059743190185429285 0.40109764424489613 0.8967900151447522
- link Link4: geometry collision box size=0.1381464667443455 0.20219850881992685 0.02124343771371673; visual box size=0.1381464667443455 0.20219850881992685 0.02124343771371673
- link Link5: geometry collision box size=0.37202815212203166 0.44585744587329 0.6800050004145273; visual box size=0.37202815212203166 0.44585744587329 0.6800050004145273
- link Link6: geometry collision box size=0.9794315229282033 0.6423910459604008 0.6182287825516497; visual box size=0.9794315229282033 0.6423910459604008 0.6182287825516497
- link Link7: geometry collision box size=0.8869800234439168 0.21520370109189535 0.14344809712418682; visual box size=0.8869800234439168 0.21520370109189535 0.14344809712418682
- link Link8: geometry collision box size=0.994230115803236 0.7663794582341745 0.11374355454843044; visual box size=0.994230115803236 0.7663794582341745 0.11374355454843044
- link Link9: geometry collision box size=0.9129008518717093 0.08740813719457352 0.815256483590447; visual box size=0.9129008518717093 0.08740813719457352 0.815256483590447
Joints:
- removed joint Link10_Link11
- removed joint Link11Link120_Link11Link121
- removed joint Link11Link121_Link12
- removed joint Link11_Link11Link120
- removed joint Link13Link140_Link14
- removed joint Link14_Link15
- removed joint Link15Link160_Link15Link161
- removed joint Link15Link161_Link16
- removed joint Link15_Link15Link160
- removed joint Link16Link170_Link16Link171
- removed joint Link16Link171_Link17
- removed joint Link16_Link16Link170
- removed joint Link17Link180_Link17Link181
- removed joint Link17Link181_Link18
- removed joint Link17_Link17Link180
- removed joint Link18Link190_Link18Link191
- removed joint Link18Link191_Link19
- removed joint Link18_Link18Link190
- removed joint Link19_Link20
- removed joint Link20Link210_Link20Link211
- removed joint Link20Link211_Link21
- removed joint Link20_Link20Link210
- removed joint Link21Link220_Link21Link221
- removed joint Link21Link221_Link22
- removed joint Link21_Link21Link220
- removed joint Link22Link230_Link23
- removed joint Link22_Link22Link230
- removed joint Link23_Link24
- removed joint Link24_Link25
- removed joint Link25Link260_Link26
- removed joint Link25_Link25Link260
- removed joint Link26Link270_Link27
- removed joint Link26_Link26Link270
- removed joint Link27Link280_Link27Link281
- removed joint Link27Link281_Link28
- removed joint Link27_Link27Link280
- removed joint Link28Link290_Link29
- removed joint Link28_Link28Link290
- removed joint Link29Link300_Link30
- removed joint Link29_Link29Link300
- removed joint Link2Link30_Link3
- removed joint Link2_Link2Link30
- removed joint Link30Link310_Link31
- removed joint Link30_Link30Link310
- removed joint Link31Link320_Link32
- removed joint Link31_Link31Link320
- removed joint Link32Link330_Link32Link331
- removed joint Link32Link331_Link33
- removed joint Link32_Link32Link330
- removed joint Link33_Link34
- removed joint Link34Link350_Link35
- removed joint Link34_Link34Link350
- removed joint Link35_Link36
- removed joint Link36_Link37
- removed joint Link37Link380_Link37Link381
- removed joint Link37Link381_Link38
- removed joint Link37_Link37Link380
- removed joint Link38Link390_Link39
- removed joint Link38_Link38Link390
- removed joint Link39Link400_Link40
- removed joint Link39_Link39Link400
- removed joint Link3_Link4
- removed joint Link40Link410_Link40Link411
- removed joint Link40Link411_Link41
- removed joint Link40_Link40Link410
- removed joint Link41Link420_Link42
- removed joint Link41_Link41Link420
- removed joint Link42_Link43
- removed joint Link43Link440_Link43Link441
- removed joint Link43Link441_Link44
- removed joint Link43_Link43Link440
- removed joint Link44_Link45
- removed joint Link45Link460_Link45Link461
- removed joint Link45Link461_Link46
- removed joint Link45_Link45Link460
- removed joint Link46Link470_Link46Link471
- removed joint Link46Link471_Link47
- removed joint Link46_Link46Link470
- removed joint Link47_Link48
- removed joint Link48Link490_Link49
- removed joint Link48_Link48Link490
- removed joint Link4Link50_Link4Link51
- removed joint Link4Link51_Link5
- removed joint Link5_Link6
- removed joint Link6Link70_Link7
- removed joint Link8Link90_Link9
- removed joint Link8_Link8Link90
- added joint Link10Link110_Link11: type revolute, parent Link10Link110, child Link11, origin xyz=0 0 0 rpy=0 0 0, axis 0 0 1, limit lower=-3.14159 upper=3.14159 effort=0.0 velocity=0.0
- added joint Link10_Link10Link110: type revolute, parent Link10, child Link10Link110, origin xyz=0.0 -0.07715142328776314 0.3065095283698596 rpy=0 0 0, axis 1 0 0, limit lower=-3.14159 upper=3.14159 effort=0.0 velocity=0.0
- added joint Link11_Link12: type revolute, parent Link11, child Link12, origin xyz=-0.11272534891551528 0.0 0.25582542107182965 rpy=0 0 0, axis 0 1 0, limit lower=-3.14159 upper=3.14159 effort=0.0 velocity=0.0
- added joint Link13Link140_Link13Link141: type revolute, parent Link13Link140, child Link13Link141, origin xyz=0 0 0 rpy=0 0 0, axis 0 1 0, limit lower=-3.14159 upper=3.14159 effort=0.0 velocity=0.0
- added joint Link13Link141_Link14: type revolute, parent Link13Link141, child Link14, origin xyz=0 0 0 rpy=0 0 0, axis 0 0 1, limit lower=-3.14159 upper=3.14159 effort=0.0 velocity=0.0
- added joint Link2_Link3: type revolute, parent Link2, child Link3, origin xyz=0.0 0.42965242144640603 -0.13026463076640454 rpy=0 0 0, axis 0 1 0, limit lower=-3.14159 upper=3.14159 effort=0.0 velocity=0.0
- added joint Link3Link40_Link4: type revolute, parent Link3Link40, child Link4, origin xyz=0 0 0 rpy=0 0 0, axis 0 0 1, limit lower=-3.14159 upper=3.14159 effort=0.0 velocity=0.0
- added joint Link3_Link3Link40: type revolute, parent Link3, child Link3Link40, origin xyz=0.0 0.0 -0.8967900151447522 rpy=0 0 0, axis 1 0 0, limit lower=-3.14159 upper=3.14159 effort=0.0 velocity=0.0
- added joint Link4Link50_Link5: type revolute, parent Link4Link50, child Link5, origin xyz=0 0 0 rpy=0 0 0, axis 1 0 0, limit lower=-3.14159 upper=3.14159 effort=0.0 velocity=0.0
- added joint Link5Link60_Link5Link61: type revolute, parent Link5Link60, child Link5Link61, origin xyz=0 0 0 rpy=0 0 0, axis 0 1 0, limit lower=-3.14159 upper=3.14159 effort=0.0 velocity=0.0
- added joint Link5Link61_Link6: type revolute, parent Link5Link61, child Link6, origin xyz=0 0 0 rpy=0 0 0, axis 1 0 0, limit lower=-3.14159 upper=3.14159 effort=0.0 velocity=0.0
- added joint Link5_Link5Link60: type revolute, parent Link5, child Link5Link60, origin xyz=0.0 0.0 0.0 rpy=0 0 0, axis 0 0 1, limit lower=-3.14159 upper=3.14159 effort=0.0 velocity=0.0
- added joint Link6Link70_Link6Link71: type revolute, parent Link6Link70, child Link6Link71, origin xyz=0 0 0 rpy=0 0 0, axis 0 0 1, limit lower=-3.14159 upper=3.14159 effort=0.0 velocity=0.0
- added joint Link6Link71_Link7: type revolute, parent Link6Link71, child Link7, origin xyz=0 0 0 rpy=0 0 0, axis 0 1 0, limit lower=-3.14159 upper=3.14159 effort=0.0 velocity=0.0
- added joint Link8_Link9: type revolute, parent Link8, child Link9, origin xyz=0.0 -0.38318972911708726 -0.05687177727421522 rpy=0 0 0, axis 0 1 0, limit lower=-3.14159 upper=3.14159 effort=0.0 velocity=0.0
- joint Link0Link10_Link1: axis 0 0 1 -> 0 1 0
- joint Link0_Link0Link10: axis 1 0 0 -> 0 0 1; origin xyz=0 0.11187622770938926 0.49385641228074606 rpy=0 0 0 -> xyz=0.0 0.0 6.8963578170033575 rpy=0 0 0
- joint Link12_Link13: axis 0 0 1 -> 0 1 0; origin xyz=0 0.34618948282382556 0 rpy=0 0 0 -> xyz=-0.16120087707033393 0.0 0.0 rpy=0 0 0
- joint Link13_Link13Link140: axis 0 1 0 -> 1 0 0; origin xyz=0 0.03163308527476549 0 rpy=0 0 0 -> xyz=-0.5818124517353301 0.0 0.0 rpy=0 0 0
- joint Link1_Link1Link20: origin xyz=0 0.18593653607767813 0 rpy=0 0 0 -> xyz=0.0 0.3498292677635674 -0.21634029522076503 rpy=0 0 0
- joint Link4_Link4Link50: origin xyz=0 0.33510369557687447 0 rpy=0 0 0 -> xyz=0.0 0.0 0.0 rpy=0 0 0
- joint Link6_Link6Link70: axis 0 0 1 -> 1 0 0; origin xyz=0 0.9465924498551117 0 rpy=0 0 0 -> xyz=-0.4897157614641017 0.0 -0.30911439127582485 rpy=0 0 0
- joint Link7_Link7Link80: origin xyz=0 0.9496152988545844 0 rpy=0 0 0 -> xyz=-0.4434900117219584 0.0 -0.07172404856209341 rpy=0 0 0
- joint Link9_Link10: origin xyz=0 0.28098950319604443 0 rpy=0 0 0 -> xyz=0.0 -0.08740813719457352 0.0 rpy=0 0 0

Commit message: 3d formation, need collision detection still" q
]\

:wq
q
"

File: body.urdf (robot description, URDF)
Before this commit: robot robot, 28 links, 27 joints
Links:
- removed link Link0Link10
- removed link Link10
- removed link Link10Link110
- removed link Link11
- removed link Link12
- removed link Link13
- removed link Link13Link140
- removed link Link13Link141
- removed link Link14
- removed link Link1Link20
- removed link Link3Link40
- removed link Link4Link50
- removed link Link5
- removed link Link5Link60
- removed link Link5Link61
- removed link Link6
- removed link Link6Link70
- removed link Link6Link71
- removed link Link7
- removed link Link7Link80
- removed link Link7Link81
- removed link Link8
- removed link Link9
- added link Cube00, mass 1; collision box size=0 0 0; visual box size=0 0 0
- added link Cube01, mass 1; collision box size=0 0 0; visual box size=0 0 0
- added link Cube02, mass 1; collision box size=0 0 0; visual box size=0 0 0
- added link Cube03, mass 1; collision box size=0 0 0; visual box size=0 0 0
- added link Cube11, mass 1; collision box size=0 0 0; visual box size=0 0 0
- added link Cube12, mass 1; collision box size=0 0 0; visual box size=0 0 0
- link Link0: geometry collision box size=0.5266267017005901 0.901621446711994 0.09959636127488258; visual box size=0.5266267017005901 0.901621446711994 0.09959636127488258
- link Link1: geometry collision box size=0.3837562745856583 0.3826171449296065 0.9836654992506204; visual box size=0.3837562745856583 0.3826171449296065 0.9836654992506204
- link Link2: geometry collision box size=0.4627510046753206 0.5671883866103837 0.8806526570193294; visual box size=0.4627510046753206 0.5671883866103837 0.8806526570193294
- link Link3: geometry collision box size=0.6364896769946986 0.5174560811395209 0.8820836098798225; visual box size=0.6364896769946986 0.5174560811395209 0.8820836098798225
- link Link4: geometry collision box size=0.026617360681923552 0.7017466726171124 0.752955965399769; visual box size=0.026617360681923552 0.7017466726171124 0.752955965399769
Joints:
- removed joint Link0Link10_Link1
- removed joint Link0_Link0Link10
- removed joint Link10Link110_Link11
- removed joint Link10_Link10Link110
- removed joint Link11_Link12
- removed joint Link12_Link13
- removed joint Link13Link140_Link13Link141
- removed joint Link13Link141_Link14
- removed joint Link13_Link13Link140
- removed joint Link1Link20_Link2
- removed joint Link1_Link1Link20
- removed joint Link2_Link3
- removed joint Link3Link40_Link4
- removed joint Link3_Link3Link40
- removed joint Link4Link50_Link5
- removed joint Link4_Link4Link50
- removed joint Link5Link60_Link5Link61
- removed joint Link5Link61_Link6
- removed joint Link5_Link5Link60
- removed joint Link6Link70_Link6Link71
- removed joint Link6Link71_Link7
- removed joint Link6_Link6Link70
- removed joint Link7Link80_Link7Link81
- removed joint Link7Link81_Link8
- removed joint Link7_Link7Link80
- removed joint Link8_Link9
- removed joint Link9_Link10
- added joint Cube00_Link1: type revolute, parent Cube00, child Link1, origin xyz=0 0 0 rpy=0 0 0, axis 0 0 1, limit lower=-3.14159 upper=3.14159 effort=0.0 velocity=0.0
- added joint Cube01_Cube11: type revolute, parent Cube01, child Cube11, origin xyz=0 0 0 rpy=0 0 0, axis 1 0 0, limit lower=-3.14159 upper=3.14159 effort=0.0 velocity=0.0
- added joint Cube02_Cube12: type revolute, parent Cube02, child Cube12, origin xyz=0 0 0 rpy=0 0 0, axis 0 1 0, limit lower=-3.14159 upper=3.14159 effort=0.0 velocity=0.0
- added joint Cube03_Link4: type revolute, parent Cube03, child Link4, origin xyz=0 0 0 rpy=0 0 0, axis 1 0 0, limit lower=-3.14159 upper=3.14159 effort=0.0 velocity=0.0
- added joint Cube11_Link2: type revolute, parent Cube11, child Link2, origin xyz=0 0 0 rpy=0 0 0, axis 0 1 0, limit lower=-3.14159 upper=3.14159 effort=0.0 velocity=0.0
- added joint Cube12_Link3: type revolute, parent Cube12, child Link3, origin xyz=0 0 0 rpy=0 0 0, axis 0 0 1, limit lower=-3.14159 upper=3.14159 effort=0.0 velocity=0.0
- added joint Link0_Cube00: type revolute, parent Link0, child Cube00, origin xyz=0.0 -0.450810723355997 3.598954092824424 rpy=0 0 0, axis 1 0 0, limit lower=-3.14159 upper=3.14159 effort=0.0 velocity=0.0
- added joint Link0_Cube01: type revolute, parent Link0, child Cube01, origin xyz=-0.26331335085029506 0.0 3.598954092824424 rpy=0 0 0, axis 0 0 1, limit lower=-3.14159 upper=3.14159 effort=0.0 velocity=0.0
- added joint Link1_Cube03: type revolute, parent Link1, child Cube03, origin xyz=-0.19187813729282915 -0.19130857246480326 0.0 rpy=0 0 0, axis 0 1 0, limit lower=-3.14159 upper=3.14159 effort=0.0 velocity=0.0
- added joint Link2_Cube02: type revolute, parent Link2, child Cube02, origin xyz=-0.2313755023376603 -0.28359419330519187 0.0 rpy=0 0 0, axis 1 0 0, limit lower=-3.14159 upper=3.14159 effort=0.0 velocity=0.0
