Commit message: optimize random creature generatio

File: body.urdf (robot description, URDF)
Before this commit: robot robot, 17 links, 16 joints
Links:
- removed link Cube01
- removed link Cube02
- removed link Cube04
- removed link Cube11
- added link Cube011, mass 1; collision box size=0 0 0; visual box size=0 0 0
- added link Cube012, mass 1; collision box size=0 0 0; visual box size=0 0 0
- added link Cube013, mass 1; collision box size=0 0 0; visual box size=0 0 0
- added link Cube03, mass 1; collision box size=0 0 0; visual box size=0 0 0
- added link Cube08, mass 1; collision box size=0 0 0; visual box size=0 0 0
- added link Cube09, mass 1; collision box size=0 0 0; visual box size=0 0 0
- added link Cube112, mass 1; collision box size=0 0 0; visual box size=0 0 0
- added link Cube113, mass 1; collision box size=0 0 0; visual box size=0 0 0
- added link Cube16, mass 1; collision box size=0 0 0; visual box size=0 0 0
- added link Cube18, mass 1; collision box size=0 0 0; visual box size=0 0 0
- added link Cube19, mass 1; collision box size=0 0 0; visual box size=0 0 0
- added link Link10, mass 1; collision box size=0.34977574689471713 0.30581691675495204 0.3794531942914196; visual box size=0.34977574689471713 0.30581691675495204 0.3794531942914196
- added link Link11, mass 1; collision box size=0.3884675497171839 0.3787876476263242 0.34929723417757275; visual box size=0.3884675497171839 0.3787876476263242 0.34929723417757275
- added link Link12, mass 1; collision box size=0.27575070990309386 0.24746958445139564 0.23280425448077963; visual box size=0.27575070990309386 0.24746958445139564 0.23280425448077963
- added link Link13, mass 1; collision box size=0.2524630524604947 0.2337335213328646 0.25822401672252965; visual box size=0.2524630524604947 0.2337335213328646 0.25822401672252965
- added link Link14, mass 1; collision box size=0.3415005016103379 0.2662874589067534 0.34573608966862707; visual box size=0.3415005016103379 0.2662874589067534 0.34573608966862707
- link Link0: geometry collision box size=0.43483496643559194 0.7030105617026852 0.3626765644989667; visual box size=0.43483496643559194 0.7030105617026852 0.3626765644989667
- link Link1: geometry collision box size=0.4282140112022309 0.4553899995207571 0.5509133817186516; visual box size=0.4282140112022309 0.4553899995207571 0.5509133817186516
- link Link2: geometry collision box size=0.41153438363246453 0.3422345202278776 0.48025420478594016; visual box size=0.41153438363246453 0.3422345202278776 0.48025420478594016
- link Link3: geometry collision box size=0.41295722041371175 0.44254821320374993 0.2206120736605998; visual box size=0.41295722041371175 0.44254821320374993 0.2206120736605998
- link Link4: geometry collision box size=0.40655958574969386 0.2558420876224621 0.40220682204037933; visual box size=0.40655958574969386 0.2558420876224621 0.40220682204037933
- link Link5: geometry collision box size=0.3084121975506855 0.30514121934273286 0.5359338039931534; visual box size=0.3084121975506855 0.30514121934273286 0.5359338039931534
- link Link6: geometry collision box size=0.3142766705004177 0.3025958806124138 0.254366656139439; visual box size=0.3142766705004177 0.3025958806124138 0.254366656139439
- link Link7: geometry collision box size=0.21658303780456586 0.34356748094693235 0.33037783403771864; visual box size=0.21658303780456586 0.34356748094693235 0.33037783403771864
- link Link8: geometry collision box size=0.4146421925559647 0.24865116125520742 0.3622100293808903; visual box size=0.4146421925559647 0.24865116125520742 0.3622100293808903
- link Link9: geometry collision box size=0.38203898823542276 0.3184698693663169 0.2922812714813132; visual box size=0.38203898823542276 0.3184698693663169 0.2922812714813132
Joints:
- removed joint Cube01_Cube11
- removed joint Cube02_Link3
- removed joint Cube04_Link5
- removed joint Cube06_Link7
- removed joint Cube11_Link2
- removed joint Link1_Cube01
- removed joint Link1_Link6
- removed joint Link2_Cube02
- removed joint Link2_Cube06
- removed joint Link3_Cube07
- removed joint Link3_Link4
- removed joint Link4_Cube04
- removed joint Link6_Link9
- added joint Cube011_Link12: type revolute, parent Cube011, child Link12, origin xyz=0 0 0 rpy=0 0 0, axis 0 0 1, limit lower=-3.14159 upper=3.14159 effort=0.0 velocity=0.0
- added joint Cube012_Cube112: type revolute, parent Cube012, child Cube112, origin xyz=0 0 0 rpy=0 0 0, axis 0 1 0, limit lower=-3.14159 upper=3.14159 effort=0.0 velocity=0.0
- added joint Cube013_Cube113: type revolute, parent Cube013, child Cube113, origin xyz=0 0 0 rpy=0 0 0, axis 0 1 0, limit lower=-3.14159 upper=3.14159 effort=0.0 velocity=0.0
- added joint Cube03_Link4: type revolute, parent Cube03, child Link4, origin xyz=0 0 0 rpy=0 0 0, axis 0 0 1, limit lower=-3.14159 upper=3.14159 effort=0.0 velocity=0.0
- added joint Cube06_Cube16: type revolute, parent Cube06, child Cube16, origin xyz=0 0 0 rpy=0 0 0, axis 0 0 1, limit lower=-3.14159 upper=3.14159 effort=0.0 velocity=0.0
- added joint Cube08_Cube18: type revolute, parent Cube08, child Cube18, origin xyz=0 0 0 rpy=0 0 0, axis 0 1 0, limit lower=-3.14159 upper=3.14159 effort=0.0 velocity=0.0
- added joint Cube09_Cube19: type revolute, parent Cube09, child Cube19, origin xyz=0 0 0 rpy=0 0 0, axis 1 0 0, limit lower=-3.14159 upper=3.14159 effort=0.0 velocity=0.0
- added joint Cube112_Link13: type revolute, parent Cube112, child Link13, origin xyz=0 0 0 rpy=0 0 0, axis 1 0 0, limit lower=-3.14159 upper=3.14159 effort=0.0 velocity=0.0
- added joint Cube113_Link14: type revolute, parent Cube113, child Link14, origin xyz=0 0 0 rpy=0 0 0, axis 0 0 1, limit lower=-3.14159 upper=3.14159 effort=0.0 velocity=0.0
- added joint Cube16_Link7: type revolute, parent Cube16, child Link7, origin xyz=0 0 0 rpy=0 0 0, axis 1 0 0, limit lower=-3.14159 upper=3.14159 effort=0.0 velocity=0.0
- added joint Cube18_Link9: type revolute, parent Cube18, child Link9, origin xyz=0 0 0 rpy=0 0 0, axis 0 0 1, limit lower=-3.14159 upper=3.14159 effort=0.0 velocity=0.0
- added joint Cube19_Link10: type revolute, parent Cube19, child Link10, origin xyz=0 0 0 rpy=0 0 0, axis 0 0 1, limit lower=-3.14159 upper=3.14159 effort=0.0 velocity=0.0
- added joint Link0_Cube03: type revolute, parent Link0, child Cube03, origin xyz=-0.21741748321779597 0.0 4.072850699188079 rpy=0 0 0, axis 1 0 0, limit lower=-3.14159 upper=3.14159 effort=0.0 velocity=0.0
- added joint Link0_Link11: type revolute, parent Link0, child Link11, origin xyz=0.21741748321779597 0.0 4.072850699188079 rpy=0 0 0, axis 0 0 1, limit lower=-3.14159 upper=3.14159 effort=0.0 velocity=0.0
- added joint Link0_Link3: type revolute, parent Link0, child Link3, origin xyz=0.0 -0.3515052808513426 4.072850699188079 rpy=0 0 0, axis 1 0 0, limit lower=-3.14159 upper=3.14159 effort=0.0 velocity=0.0
- added joint Link11_Cube013: type revolute, parent Link11, child Cube013, origin xyz=0.19423377485859195 0.0 0.17464861708878637 rpy=0 0 0, axis 1 0 0, limit lower=-3.14159 upper=3.14159 effort=0.0 velocity=0.0
- added joint Link1_Cube06: type revolute, parent Link1, child Cube06, origin xyz=0.0 0.4553899995207571 0.0 rpy=0 0 0, axis 0 1 0, limit lower=-3.14159 upper=3.14159 effort=0.0 velocity=0.0
- added joint Link1_Link2: type revolute, parent Link1, child Link2, origin xyz=0.0 0.22769499976037855 -0.2754566908593258 rpy=0 0 0, axis 0 1 0, limit lower=-3.14159 upper=3.14159 effort=0.0 velocity=0.0
- added joint Link1_Link5: type revolute, parent Link1, child Link5, origin xyz=0.0 0.22769499976037855 0.2754566908593258 rpy=0 0 0, axis 0 0 1, limit lower=-3.14159 upper=3.14159 effort=0.0 velocity=0.0
- added joint Link2_Cube011: type revolute, parent Link2, child Cube011, origin xyz=0.0 -0.1711172601139388 -0.24012710239297008 rpy=0 0 0, axis 0 1 0, limit lower=-3.14159 upper=3.14159 effort=0.0 velocity=0.0
- added joint Link2_Cube012: type revolute, parent Link2, child Cube012, origin xyz=-0.20576719181623226 0.0 -0.24012710239297008 rpy=0 0 0, axis 0 0 1, limit lower=-3.14159 upper=3.14159 effort=0.0 velocity=0.0
- added joint Link2_Cube08: type revolute, parent Link2, child Cube08, origin xyz=0.20576719181623226 0.0 -0.24012710239297008 rpy=0 0 0, axis 1 0 0, limit lower=-3.14159 upper=3.14159 effort=0.0 velocity=0.0
- added joint Link3_Link6: type revolute, parent Link3, child Link6, origin xyz=0.20647861020685587 -0.22127410660187496 0.0 rpy=0 0 0, axis 0 0 1, limit lower=-3.14159 upper=3.14159 effort=0.0 velocity=0.0
- added joint Link4_Cube09: type revolute, parent Link4, child Cube09, origin xyz=-0.20327979287484693 0.0 0.20110341102018967 rpy=0 0 0, axis 0 1 0, limit lower=-3.14159 upper=3.14159 effort=0.0 velocity=0.0
- added joint Link5_Cube07: type revolute, parent Link5, child Cube07, origin xyz=0.0 0.0 0.5359338039931534 rpy=0 0 0, axis 0 1 0, limit lower=-3.14159 upper=3.14159 effort=0.0 velocity=0.0
- joint Cube07_Cube17: axis 0 1 0 -> 1 0 0
- joint Cube17_Link8: axis 1 0 0 -> 0 0 1
- joint Link0_Link1: axis 0 1 0 -> 1 0 0; origin xyz=0.3403771055665182 0.0 3.0668260537413468 rpy=0 0 0 -> xyz=0.0 0.3515052808513426 4.072850699188079 rpy=0 0 0

Commit message: add mutations

File: body.urdf (robot description, URDF)
Before this commit: robot robot, 29 links, 28 joints
Links:
- removed link Cube011
- removed link Cube012
- removed link Cube013
- removed link Cube07
- removed link Cube08
- removed link Cube09
- removed link Cube112
- removed link Cube113
- removed link Cube16
- removed link Cube17
- removed link Cube18
- removed link Cube19
- removed link Link10
- removed link Link11
- removed link Link12
- removed link Link13
- removed link Link14
- added link Cube02, mass 1; collision box size=0 0 0; visual box size=0 0 0
- added link Cube04, mass 1; collision box size=0 0 0; visual box size=0 0 0
- added link Cube13, mass 1; collision box size=0 0 0; visual box size=0 0 0
- added link Cube14, mass 1; collision box size=0 0 0; visual box size=0 0 0
- link Link0: geometry collision box size=0.7538483094758679 0.545200814240463 0.33146565373824055; visual box size=0.7538483094758679 0.545200814240463 0.33146565373824055
- link Link1: geometry collision box size=0.7504010688165668 0.34931593646393666 0.6435115141356299; visual box size=0.7504010688165668 0.34931593646393666 0.6435115141356299
- link Link2: geometry collision box size=0.7075063339719769 0.23920108892450234 0.24708405388927623; visual box size=0.7075063339719769 0.23920108892450234 0.24708405388927623
- link Link3: geometry collision box size=0.32234584787606657 0.20446130934221626 0.4117713644617902; visual box size=0.32234584787606657 0.20446130934221626 0.4117713644617902
- link Link4: geometry collision box size=0.44187555566416015 0.31061645345846955 0.3314403242905859; visual box size=0.44187555566416015 0.31061645345846955 0.3314403242905859
- link Link5: geometry collision box size=0.7026741207950489 0.39570036244214357 0.3632533494834495; visual box size=0.7026741207950489 0.39570036244214357 0.3632533494834495
- link Link6: geometry collision box size=0.353243847350854 0.2381685246440954 0.5817035716138588; visual box size=0.353243847350854 0.2381685246440954 0.5817035716138588
- link Link7: geometry collision box size=0.6596725785315147 0.5962584766690391 0.42571971225040395; visual box size=0.6596725785315147 0.5962584766690391 0.42571971225040395
- link Link8: geometry collision box size=0.47968146787892385 0.5286510378591887 0.4617670548492693; visual box size=0.47968146787892385 0.5286510378591887 0.4617670548492693
- link Link9: geometry collision box size=0.33972993828810283 0.22298208696737973 0.29712781525883636; visual box size=0.33972993828810283 0.22298208696737973 0.29712781525883636
Joints:
- removed joint Cube011_Link12
- removed joint Cube012_Cube112
- removed joint Cube013_Cube113
- removed joint Cube03_Link4
- removed joint Cube06_Cube16
- removed joint Cube07_Cube17
- removed joint Cube08_Cube18
- removed joint Cube09_Cube19
- removed joint Cube112_Link13
- removed joint Cube113_Link14
- removed joint Cube16_Link7
- removed joint Cube17_Link8
- removed joint Cube18_Link9
- removed joint Cube19_Link10
- removed joint Link0_Cube03
- removed joint Link0_Link11
- removed joint Link0_Link3
- removed joint Link11_Cube013
- removed joint Link1_Cube06
- removed joint Link1_Link5
- removed joint Link2_Cube011
- removed joint Link2_Cube012
- removed joint Link2_Cube08
- removed joint Link3_Link6
- removed joint Link4_Cube09
- removed joint Link5_Cube07
- added joint Cube02_Link3: type revolute, parent Cube02, child Link3, origin xyz=0 0 0 rpy=0 0 0, axis 1 0 0, limit lower=-3.14159 upper=3.14159 effort=0.0 velocity=0.0
- added joint Cube03_Cube13: type revolute, parent Cube03, child Cube13, origin xyz=0 0 0 rpy=0 0 0, axis 1 0 0, limit lower=-3.14159 upper=3.14159 effort=0.0 velocity=0.0
- added joint Cube04_Cube14: type revolute, parent Cube04, child Cube14, origin xyz=0 0 0 rpy=0 0 0, axis 0 0 1, limit lower=-3.14159 upper=3.14159 effort=0.0 velocity=0.0
- added joint Cube06_Link7: type revolute, parent Cube06, child Link7, origin xyz=0 0 0 rpy=0 0 0, axis 1 0 0, limit lower=-3.14159 upper=3.14159 effort=0.0 velocity=0.0
- added joint Cube13_Link4: type revolute, parent Cube13, child Link4, origin xyz=0 0 0 rpy=0 0 0, axis 0 0 1, limit lower=-3.14159 upper=3.14159 effort=0.0 velocity=0.0
- added joint Cube14_Link5: type revolute, parent Cube14, child Link5, origin xyz=0 0 0 rpy=0 0 0, axis 0 1 0, limit lower=-3.14159 upper=3.14159 effort=0.0 velocity=0.0
- added joint Link0_Cube04: type revolute, parent Link0, child Cube04, origin xyz=-0.37692415473793395 0.0 3.223675879264918 rpy=0 0 0, axis 1 0 0, limit lower=-3.14159 upper=3.14159 effort=0.0 velocity=0.0
- added joint Link0_Link8: type revolute, parent Link0, child Link8, origin xyz=0.0 -0.2726004071202315 3.223675879264918 rpy=0 0 0, axis 1 0 0, limit lower=-3.14159 upper=3.14159 effort=0.0 velocity=0.0
- added joint Link1_Cube03: type revolute, parent Link1, child Cube03, origin xyz=0.3752005344082834 0.0 0.32175575706781495 rpy=0 0 0, axis 0 1 0, limit lower=-3.14159 upper=3.14159 effort=0.0 velocity=0.0
- added joint Link1_Link6: type revolute, parent Link1, child Link6, origin xyz=0.3752005344082834 0.0 -0.32175575706781495 rpy=0 0 0, axis 0 0 1, limit lower=-3.14159 upper=3.14159 effort=0.0 velocity=0.0
- added joint Link2_Cube02: type revolute, parent Link2, child Cube02, origin xyz=0.7075063339719769 0.0 0.0 rpy=0 0 0, axis 0 0 1, limit lower=-3.14159 upper=3.14159 effort=0.0 velocity=0.0
- added joint Link3_Link9: type revolute, parent Link3, child Link9, origin xyz=0.16117292393803329 0.0 -0.2058856822308951 rpy=0 0 0, axis 0 1 0, limit lower=-3.14159 upper=3.14159 effort=0.0 velocity=0.0
- added joint Link5_Cube06: type revolute, parent Link5, child Cube06, origin xyz=-0.7026741207950489 0.0 0.0 rpy=0 0 0, axis 0 0 1, limit lower=-3.14159 upper=3.14159 effort=0.0 velocity=0.0
- joint Link0_Link1: origin xyz=0.0 0.3515052808513426 4.072850699188079 rpy=0 0 0 -> xyz=0.37692415473793395 0.0 3.223675879264918 rpy=0 0 0
- joint Link1_Link2: origin xyz=0.0 0.22769499976037855 -0.2754566908593258 rpy=0 0 0 -> xyz=0.7504010688165668 0.0 0.0 rpy=0 0 0
